File: pcb/IGG1_OctoDriver.kicad_sch (KiCad schematic)
At the start: 91 parts, among them J1 Conn_01x01, J10 Conn_01x01, J11 Conn_01x01, J12 Conn_01x01, J13 Conn_01x01, J14 Conn_01x01, J15 Conn_01x01, J16 Conn_01x01, J17 Conn_01x01, J18 Conn_01x01, J19 TEST_1P, J2 Conn_01x08, J3 Conn_01x08, J4 Conn_01x01, J5 Conn_01x08, J6 Conn_01x08, J7 Conn_01x08, J8 Conn_01x08, J9 Conn_01x01, Q1 Q_NPN_BEC, Q10 Q_NPN_BEC, Q11 Q_NPN_BEC, Q12 Q_NPN_BEC, Q13 Q_NPN_BEC, Q14 Q_NPN_BEC, Q15 Q_NPN_BEC, Q16 Q_NPN_BEC, Q17 Q_NPN_BEC, Q18 Q_NPN_BEC, Q19 Q_NPN_BEC, Q20 Q_NPN_BEC, Q21 Q_NPN_BEC, Q22 Q_NPN_BEC, Q23 Q_NPN_BEC, Q24 Q_NPN_BEC, Q9 Q_NPN_BEC, U10 74LS541, U9 74LS541

Commit message: Added kathode driver
Parts:
- removed C10, C9: 100n, Capacitors_SMD:C_1206, symbol IGG1_OctoDriver-rescue:C
- removed J3, J6, J7, J8: Conn_01x08, footprints:Pin_Header_1x08_Pitch1.27mm_SMD, symbol IGG1_OctoDriver-rescue:Conn_01x08
- removed U10, U9: 74LS541, Housings_SSOP:TSSOP-20_4.4x6.5mm_Pitch0.65mm, symbol IGG1_OctoDriver-rescue:74LS541
- added C12, C14, C16, C18, C19, C21, C22, C23, C24, C25: 100nf, Capacitor_SMD:C_0603_1608Metric, symbol Device:C
- added C13, C15: 4.7pF, Capacitor_SMD:C_0603_1608Metric, symbol Device:C
- added C17, C20: 1uf, Capacitor_SMD:C_0603_1608Metric, symbol Device:C
- added C2, C3, C4, C5, C6, C7, C8: 1n, Capacitors_SMD:C_1206, symbol IGG1_OctoDriver-rescue:C
- added D18: D, Diode_SMD:D_SMA, symbol Device:D
- added H1, H2, H3, H4: H, MountingHole:MountingHole_3.2mm_M3_DIN965_Pad, symbol Mechanical:MountingHole_Pad
- added J21: USB_C_Receptacle_USB2.0, Connector_USB:USB_C_Receptacle_HRO_TYPE-C-31-M-12, symbol Connector:USB_C_Receptacle_USB2.0
- added J22: Conn_ARM_SWD_TagConnect_TC2030-NL, Connector:Tag-Connect_TC2030-IDC-NL_2x03_P1.27mm_Vertical, symbol Connector:Conn_ARM_SWD_TagConnect_TC2030-NL
- added Q2, Q3, Q4, Q5, Q6, Q7, Q8: Q_NPN_BEC, TO_SOT_Packages_SMD:SOT-23, symbol IGG1_OctoDriver-rescue:Q_NPN_BEC
- added R10, R12, R14, R16, R3, R5, R7: 4.7K, Resistors_SMD:R_1206, symbol IGG1_OctoDriver-rescue:R
- added R11, R13, R15, R2, R4, R6, R8: 220K, Resistors_SMD:R_1206, symbol IGG1_OctoDriver-rescue:R
- added R49, R52: 1K, Resistor_SMD:R_0603_1608Metric, symbol Device:R
- added R50: 10K, Resistor_SMD:R_0603_1608Metric, symbol Device:R
- added R51: DNP, Resistor_SMD:R_0603_1608Metric, symbol Device:R
- added R53, R54: 27, Resistor_SMD:R_0603_1608Metric, symbol Device:R
- added R55, R56: 5k1, Resistor_SMD:R_0603_1608Metric, symbol Device:R
- added SW1: SW_Push, Button_Switch_SMD:SW_SPST_TL3342, symbol Switch:SW_Push
- added U1: W25Q128JVS, Package_SO:SOIC-8_5.23x5.23mm_P1.27mm, symbol Memory_Flash:W25Q128JVS
- added U2: RP2040, MCU_RaspberryPi_and_Boards:RP2040-QFN-56, symbol MCU_RaspberryPi_and_Boards:RP2040
- added Y1: 12M, Crystal:Crystal_SMD_5032-2Pin_5.0x3.2mm, symbol Device:Crystal
- Q17, Q9: LCSC (none) -> C151355
Connections:
- net AI0: now also U2.2 (GPIO0)
- net AI1: now also U2.3 (GPIO1)
- net AI2: now also U2.4 (GPIO2)
- net AI3: now also U2.5 (GPIO3)
- net AI4: now also U2.6 (GPIO4)
- net AI5: now also U2.7 (GPIO5)
- net AI6: now also U2.8 (GPIO6)
- net AI7: now also U2.9 (GPIO7)
- net GND: now also C12.2, C13.2, C14.2, C15.2, C16.2, C17.2, C18.2, C19.2, C20.2, C21.2, C22.2, C23.2, C24.2, C25.2, H1.1, H2.1, H3.1, H4.1, J21.A1 (GND), J21.A12 (GND), J21.B1 (GND), J21.B12 (GND), J21.S1 (SHIELD), J22.5 (GND), Q2.2 (E), Q3.2 (E), R55.1, R56.1, SW1.2, U1.4 (GND), U2.19 (TESTEN), U2.57 (GND); no longer Q17.2 (E), Q9.2 (E)
- net HT: now also Q17.3 (C), Q9.3 (C), Q4.3 (C), Q5.3 (C), Q6.3 (C), Q7.3 (C), Q8.3 (C), R10.1, R11.1, R12.1, R13.1, R14.1, R15.1, R16.1, R2.1, R3.1, R4.1, R5.1, R6.1, R7.1, R8.1
- net KI0: now also U2.16 (GPIO13)
- net KI1: now also U2.17 (GPIO14)
- net KI2: now also U2.18 (GPIO15)
- net KI3: now also U2.27 (GPIO16)
- net KI4: now also U2.28 (GPIO17)
- net KI5: now also U2.29 (GPIO18)
- net KI6: now also U2.30 (GPIO19)
- net KI7: now also U2.31 (GPIO20)
- net KO0: now also Q3.3 (C); no longer Q17.3 (C)
- net at D1.1 (K), Q1.1 (B), R1.2: now also Q2.3 (C); no longer Q9.3 (C)
- net at R17.1: now also Q2.1 (B); no longer Q9.1 (B)
- net at R41.1: now also Q3.1 (B); no longer Q17.1 (B)
- net at D4.1 (K), R20.2: now also C2.1
- net at D3.1 (K), Q10.3 (C): now also Q4.1 (B), R2.2
- net at D6.1 (K), R22.2: now also C3.1
- net at D5.1 (K), Q11.3 (C): now also Q5.1 (B), R4.2
- net at D8.1 (K), R24.2: now also C4.1
- net at D7.1 (K), Q12.3 (C): now also Q6.1 (B), R6.2
- net at D10.1 (K), R26.2: now also C5.1
- net at D9.1 (K), Q13.3 (C): now also Q7.1 (B), R8.2
- net at D12.1 (K), R28.2: now also C6.1
- net at D11.1 (K), Q14.3 (C): now also Q8.1 (B), R11.2
- net at D14.1 (K), R30.2: now also C7.1
- net at D13.1 (K), Q15.3 (C): now also Q9.1 (B), R13.2
- net at D16.1 (K), R32.2: now also C8.1
- net at D15.1 (K), Q16.3 (C): now also Q17.1 (B), R15.2
- net at D5.2 (A): now also C3.2, Q5.2 (E)
- net at D10.2 (A): now also R10.2
- net at D9.2 (A): now also C5.2, Q7.2 (E)
- net at D13.2 (A): now also Q9.2 (E), C7.2
- net at D6.2 (A): now also R5.2
- net at D15.2 (A): now also Q17.2 (E), C8.2
- net at D8.2 (A): now also R7.2
- net at D16.2 (A): now also R16.2
- net at D3.2 (A): now also C2.2, Q4.2 (E)
- net at D7.2 (A): now also C4.2, Q6.2 (E)
- net at D12.2 (A): now also R12.2
- net at D4.2 (A): now also R3.2
- net at D14.2 (A): now also R14.2
- net at D11.2 (A): now also C6.2, Q8.2 (E)
- new net: R54.1, U2.46 (USB_DM)
- new net: C15.1, U2.21 (XOUT), Y1.2
- new net: C13.1, R52.1, Y1.1
- new net: R52.2, U2.20 (XIN)
- new net: D18.2 (A), J21.A4 (VBUS), J21.A9 (VBUS), J21.B4 (VBUS), J21.B9 (VBUS)
- new net: R49.2, R51.2, U1.1 (~{CS}), U2.56 (QSPI_SS)
- new net: R53.1, U2.47 (USB_DP)
- new net: J22.4 (SWCLK), U2.24 (SWCLK)
- new net: J22.2 (SWDIO), U2.25 (SWD)
- new net: U1.7 (IO3), U2.51 (QSPI_SD3)
- new net: U1.6 (CLK), U2.52 (QSPI_SCLK)
- new net: U1.5 (DI(IO0)), U2.53 (QSPI_SD0)
- new net: U1.3 (IO2), U2.54 (QSPI_SD2)
- new net: U1.2 (DO(IO1)), U2.55 (QSPI_SD1)
- new net: J21.A5 (CC1), R56.2
- new net: J21.B5 (CC2), R55.2
- new net +12V: D18.1 (K)
- new net +1V1: C14.1, C16.1, C17.1, U2.23 (DVDD), U2.45 (VREG_VOUT), U2.50 (DVDD)
- new net +3V3: C12.1, C18.1, C19.1, C20.1, C21.1, C22.1, C23.1, C24.1, C25.1, J22.1 (VCC), R50.2, R51.1, U1.8 (VCC), U2.1 (IOVDD), U2.10 (IOVDD), U2.22 (IOVDD), U2.33 (IOVDD), U2.42 (IOVDD), U2.43 (ADC_AVDD), U2.44 (VREG_IN), U2.48 (USB_VDD), U2.49 (IOVDD)
- new net AI10: U2.13 (GPIO10)
- new net AI11: U2.14 (GPIO11)
- new net AI12: U2.15 (GPIO12)
- new net AI8: U2.11 (GPIO8)
- new net AI9: U2.12 (GPIO9)
- new net KI10: U2.35 (GPIO23)
- new net KI11: U2.36 (GPIO24)
- new net KI12: U2.37 (GPIO25)
- new net KI8: U2.32 (GPIO21)
- new net KI9: U2.34 (GPIO22)
- new net RST: J22.3 (~{RESET}), R50.1, U2.26 (RUN)
- new net USB_D+: J21.A6 (D+), J21.B6 (D+), R53.2
- new net USB_D-: J21.A7 (D-), J21.B7 (D-), R54.2
- new net ~{USB_BOOT}: R49.1, SW1.1

Commit message: Schematic almost done for anode
Parts:
- removed C1, C2, C3, C4, C5, C6, C7, C8: 1n, Capacitors_SMD:C_1206, symbol IGG1_OctoDriver-rescue:C
- removed D1, D10, D11, D12, D13, D14, D15, D16, D2, D3, D4, D5, D6, D7, D8, D9: D, Diode_SMD:D_SOD-323, symbol Device:D
- removed J1, J10, J11, J12, J13, J14, J15, J16, J17, J18, J4, J9: Conn_01x01, Pin_Headers:Pin_Header_Straight_1x01_Pitch2.54mm, symbol IGG1_OctoDriver-rescue:Conn_01x01
- removed J19: TEST_1P, footprints:via, symbol IGG1_OctoDriver-rescue:TEST_1P
- removed J2, J5: Conn_01x08, footprints:Pin_Header_21x04_Pitch2.54mm_SMD_2sides, symbol IGG1_OctoDriver-rescue:Conn_01x08
- removed Q1, Q10, Q11, Q12, Q13, Q14, Q15, Q16, Q17, Q18, Q19, Q2, Q20, Q21, Q22, Q23, Q24, Q3, Q4, Q5, Q6, Q7, Q8, Q9: Q_NPN_BEC, TO_SOT_Packages_SMD:SOT-23, symbol IGG1_OctoDriver-rescue:Q_NPN_BEC
- removed R1, R11, R13, R15, R2, R33, R34, R35, R36, R37, R38, R39, R4, R40, R6, R8: 220K, Resistors_SMD:R_1206, symbol IGG1_OctoDriver-rescue:R
- removed R10, R12, R14, R16, R3, R5, R7, R9: 4.7K, Resistors_SMD:R_1206, symbol IGG1_OctoDriver-rescue:R
- removed R17, R19, R21, R23, R25, R27, R29, R31, R41, R42, R43, R44, R45, R46, R47, R48: 10K, Resistors_SMD:R_1206, symbol IGG1_OctoDriver-rescue:R
- removed R18, R20, R22, R24, R26, R28, R30, R32: 100K, Resistors_SMD:R_1206, symbol IGG1_OctoDriver-rescue:R
- added JP1, JP2, JP3, JP4, JP5, JP6, JP7: Jumper_2_Open, symbol Jumper:Jumper_2_Open
- added U10, U11, U4, U5, U6, U7, U8, U9: 74AHCT595, symbol 74xx:74AHCT595
- added U3: ~, symbol IGG1:IGG1-64
Connections:
- net AI1: now also U4.15 (QA); no longer U2.3 (GPIO1)
- net AI10: now also U5.1 (QB); no longer U2.13 (GPIO10)
- net AI11: now also U5.2 (QC); no longer U2.14 (GPIO11)
- net AI12: now also U5.3 (QD); no longer U2.15 (GPIO12)
- net AI2: now also U4.1 (QB); no longer U2.4 (GPIO2)
- net AI3: now also U4.2 (QC); no longer U2.5 (GPIO3)
- net AI4: now also U4.3 (QD); no longer U2.6 (GPIO4)
- net AI5: now also U4.4 (QE); no longer U2.7 (GPIO5)
- net AI6: now also U4.5 (QF); no longer U2.8 (GPIO6)
- net AI7: now also U4.6 (QG); no longer U2.9 (GPIO7)
- net AI8: now also U4.7 (QH); no longer U2.11 (GPIO8)
- net AI9: now also U5.15 (QA); no longer U2.12 (GPIO9)
- net AO1: now also U3.1
- net AO2: now also U3.2
- net AO3: now also U3.3
- net AO4: now also U3.4
- net AO5: now also U3.5
- net AO6: now also U3.6
- net AO7: now also U3.7
- net GND: now also U10.8 (GND), U11.8 (GND), U4.8 (GND), U5.8 (GND), U6.8 (GND), U7.8 (GND), U8.8 (GND), U9.8 (GND)
- net AI0 renamed SR_D1
- net SR_D1: now also U4.14 (SER)
- net KI0: no longer names the net of U2.16 (GPIO13)
- net KI1: no longer names the net of U2.17 (GPIO14)
- net KI10: no longer names the net of U2.35 (GPIO23)
- net KI11: no longer names the net of U2.36 (GPIO24)
- net KI12: no longer names the net of U2.37 (GPIO25)
- net KI2: no longer names the net of U2.18 (GPIO15)
- net KI3: no longer names the net of U2.27 (GPIO16)
- net KI4: no longer names the net of U2.28 (GPIO17)
- net KI5: no longer names the net of U2.29 (GPIO18)
- net KI6: no longer names the net of U2.30 (GPIO19)
- net KI7: no longer names the net of U2.31 (GPIO20)
- net KI8: no longer names the net of U2.32 (GPIO21)
- net KI9: no longer names the net of U2.34 (GPIO22)
- new net: JP4.1 (A), U7.9 (QH')
- new net: JP1.1 (A), U4.9 (QH')
- new net: JP2.1 (A), U5.9 (QH')
- new net: JP3.1 (A), U6.9 (QH')
- new net: JP7.1 (A), U10.9 (QH')
- new net: JP5.1 (A), U8.9 (QH')
- new net: JP6.1 (A), U9.9 (QH')
- new net +5V: U10.16 (VCC), U11.16 (VCC), U4.16 (VCC), U5.16 (VCC), U6.16 (VCC), U7.16 (VCC), U8.16 (VCC), U9.16 (VCC)
- new net AI13: U5.4 (QE)
- new net AI14: U5.5 (QF)
- new net AI15: U5.6 (QG)
- new net AI16: U5.7 (QH)
- new net AI17: U6.15 (QA)
- new net AI18: U6.1 (QB)
- new net AI19: U6.2 (QC)
- new net AI20: U6.3 (QD)
- new net AI21: U6.4 (QE)
- new net AI22: U6.5 (QF)
- new net AI23: U6.6 (QG)
- new net AI24: U6.7 (QH)
- new net AI25: U7.15 (QA)
- new net AI26: U7.1 (QB)
- new net AI27: U7.2 (QC)
- new net AI28: U7.3 (QD)
- new net AI29: U7.4 (QE)
- new net AI30: U7.5 (QF)
- new net AI31: U7.6 (QG)
- new net AI32: U7.7 (QH)
- new net AI33: U8.15 (QA)
- new net AI34: U8.1 (QB)
- new net AI35: U8.2 (QC)
- new net AI36: U8.3 (QD)
- new net AI37: U8.4 (QE)
- new net AI38: U8.5 (QF)
- new net AI39: U8.6 (QG)
- new net AI40: U8.7 (QH)
- new net AI41: U9.15 (QA)
- new net AI42: U9.1 (QB)
- new net AI43: U9.2 (QC)
- new net AI44: U9.3 (QD)
- new net AI45: U9.4 (QE)
- new net AI46: U9.5 (QF)
- new net AI47: U9.6 (QG)
- new net AI48: U9.7 (QH)
- new net AI49: U10.15 (QA)
- new net AI50: U10.1 (QB)
- new net AI51: U10.2 (QC)
- new net AI52: U10.3 (QD)
- new net AI53: U10.4 (QE)
- new net AI54: U10.5 (QF)
- new net AI55: U10.6 (QG)
- new net AI56: U10.7 (QH)
- new net AI57: U11.15 (QA)
- new net AI58: U11.1 (QB)
- new net AI59: U11.2 (QC)
- new net AI60: U11.3 (QD)
- new net AI61: U11.4 (QE)
- new net AI62: U11.5 (QF)
- new net AI63: U11.6 (QG)
- new net AI64: U11.7 (QH)
- new net AO10: U3.10
- new net AO11: U3.11
- new net AO12: U3.12
- new net AO13: U3.13
- new net AO14: U3.14
- new net AO15: U3.15
- new net AO16: U3.16
- new net AO17: U3.17
- new net AO18: U3.18
- new net AO19: U3.19
- new net AO20: U3.20
- new net AO21: U3.21
- new net AO22: U3.22
- new net AO23: U3.23
- new net AO24: U3.24
- new net AO25: U3.25
- new net AO26: U3.26
- new net AO27: U3.27
- new net AO28: U3.28
- new net AO29: U3.29
- new net AO30: U3.30
- new net AO31: U3.31
- new net AO32: U3.32
- new net AO33: U3.33
- new net AO34: U3.34
- new net AO35: U3.35
- new net AO36: U3.36
- new net AO37: U3.37
- new net AO38: U3.38
- new net AO39: U3.39
- new net AO40: U3.40
- new net AO41: U3.41
- new net AO42: U3.42
- new net AO43: U3.43
- new net AO44: U3.44
- new net AO45: U3.45
- new net AO46: U3.46
- new net AO47: U3.47
- new net AO48: U3.48
- new net AO49: U3.49
- new net AO50: U3.50
- new net AO51: U3.51
- new net AO52: U3.52
- new net AO53: U3.53
- new net AO54: U3.54
- new net AO55: U3.55
- new net AO56: U3.56
- new net AO57: U3.57
- new net AO58: U3.58
- new net AO59: U3.59
- new net AO60: U3.60
- new net AO61: U3.61
- new net AO62: U3.62
- new net AO63: U3.63
- new net AO64: U3.64
- new net AO8: U3.8
- new net AO9: U3.9
- new net SR_D2: JP1.2 (B), U2.3 (GPIO1), U5.14 (SER)
- new net SR_D3: JP2.2 (B), U2.4 (GPIO2), U6.14 (SER)
- new net SR_D4: JP3.2 (B), U2.5 (GPIO3), U7.14 (SER)
- new net SR_D5: JP4.2 (B), U2.6 (GPIO4), U8.14 (SER)
- new net SR_D6: JP5.2 (B), U2.7 (GPIO5), U9.14 (SER)
- new net SR_D7: JP6.2 (B), U10.14 (SER), U2.8 (GPIO6)
- new net SR_D8: JP7.2 (B), U11.14 (SER), U2.9 (GPIO7)
- new net SR_SHCP: U10.11 (SRCLK), U11.11 (SRCLK), U4.11 (SRCLK), U5.11 (SRCLK), U6.11 (SRCLK), U7.11 (SRCLK), U8.11 (SRCLK), U9.11 (SRCLK)
- new net SR_STCP: U10.12 (RCLK), U11.12 (RCLK), U4.12 (RCLK), U5.12 (RCLK), U6.12 (RCLK), U7.12 (RCLK), U8.12 (RCLK), U9.12 (RCLK)
- new net ~SR_MC: U10.10 (~{SRCLR}), U11.10 (~{SRCLR}), U4.10 (~{SRCLR}), U5.10 (~{SRCLR}), U6.10 (~{SRCLR}), U7.10 (~{SRCLR}), U8.10 (~{SRCLR}), U9.10 (~{SRCLR})
- new net ~SR_OE: U10.13 (~{OE}), U11.13 (~{OE}), U4.13 (~{OE}), U5.13 (~{OE}), U6.13 (~{OE}), U7.13 (~{OE}), U8.13 (~{OE}), U9.13 (~{OE})
Other:
- added sheet Anode (anode.kicad_sch)
- added sheet Anode1 (anode.kicad_sch)
- added sheet Anode10 (anode.kicad_sch)
- added sheet Anode11 (anode.kicad_sch)
- added sheet Anode12 (anode.kicad_sch)
- added sheet Anode13 (anode.kicad_sch)
- added sheet Anode14 (anode.kicad_sch)
- added sheet Anode15 (anode.kicad_sch)
- added sheet Anode16 (anode.kicad_sch)
- added sheet Anode17 (anode.kicad_sch)
- added sheet Anode18 (anode.kicad_sch)
- added sheet Anode19 (anode.kicad_sch)
- added sheet Anode2 (anode.kicad_sch)
- added sheet Anode20 (anode.kicad_sch)
- added sheet Anode21 (anode.kicad_sch)
- added sheet Anode22 (anode.kicad_sch)
- added sheet Anode23 (anode.kicad_sch)
- added sheet Anode24 (anode.kicad_sch)
- added sheet Anode25 (anode.kicad_sch)
- added sheet Anode26 (anode.kicad_sch)
- added sheet Anode27 (anode.kicad_sch)
- added sheet Anode28 (anode.kicad_sch)
- added sheet Anode29 (anode.kicad_sch)
- added sheet Anode3 (anode.kicad_sch)
- added sheet Anode30 (anode.kicad_sch)
- added sheet Anode31 (anode.kicad_sch)
- added sheet Anode32 (anode.kicad_sch)
- added sheet Anode33 (anode.kicad_sch)
- added sheet Anode34 (anode.kicad_sch)
- added sheet Anode35 (anode.kicad_sch)
- added sheet Anode36 (anode.kicad_sch)
- added sheet Anode37 (anode.kicad_sch)
- added sheet Anode38 (anode.kicad_sch)
- added sheet Anode39 (anode.kicad_sch)
- added sheet Anode4 (anode.kicad_sch)
- added sheet Anode40 (anode.kicad_sch)
- added sheet Anode41 (anode.kicad_sch)
- added sheet Anode42 (anode.kicad_sch)
- added sheet Anode43 (anode.kicad_sch)
- added sheet Anode44 (anode.kicad_sch)
- added sheet Anode45 (anode.kicad_sch)
- added sheet Anode46 (anode.kicad_sch)
- added sheet Anode47 (anode.kicad_sch)
- added sheet Anode48 (anode.kicad_sch)
- added sheet Anode49 (anode.kicad_sch)
- added sheet Anode5 (anode.kicad_sch)
- added sheet Anode50 (anode.kicad_sch)
- added sheet Anode51 (anode.kicad_sch)
- added sheet Anode52 (anode.kicad_sch)
- added sheet Anode53 (anode.kicad_sch)
- added sheet Anode54 (anode.kicad_sch)
- added sheet Anode55 (anode.kicad_sch)
- added sheet Anode56 (anode.kicad_sch)
- added sheet Anode57 (anode.kicad_sch)
- added sheet Anode58 (anode.kicad_sch)
- added sheet Anode59 (anode.kicad_sch)
- added sheet Anode6 (anode.kicad_sch)
- added sheet Anode60 (anode.kicad_sch)
- added sheet Anode61 (anode.kicad_sch)
- added sheet Anode7 (anode.kicad_sch)
- added sheet Anode8 (anode.kicad_sch)
- added sheet Anode9 (anode.kicad_sch)

Commit message: Schematic of anode basically done, started layout
Parts:
- added C1, C10, C11, C12, C13, C14, C2, C3, C4, C5, C7, C8, C9: 1u, Capacitor_SMD:C_0603_1608Metric, symbol Device:C
- added C15, C6: 22u, Capacitor_SMD:C_1206_3216Metric, symbol Device:C
- added D1, D2, D3, D4, D5, D6: SK6812, LED_SMD:LED_SK6812MINI_PLCC4_3.5x3.5mm_P1.75mm, symbol LED:SK6812
- added D7: D, Diode_SMD:D_SMA, symbol Device:D
- added J1, J4: Conn_01x02, Connector_JST:JST_XH_B2B-XH-AM_1x02_P2.50mm_Vertical, symbol Connector_Generic:Conn_01x02
- added J2: Conn_01x05, Connector_JST:JST_XH_B5B-XH-AM_1x05_P2.50mm_Vertical, symbol Connector_Generic:Conn_01x05
- added J3: Conn_01x04, Connector_JST:JST_XH_B4B-XH-AM_1x04_P2.50mm_Vertical, symbol Connector_Generic:Conn_01x04
- added L1: 22uH, Inductor_SMD:L_Chilisin_BMRF00101040, symbol Device:L
- added R1: 47K, Resistor_SMD:R_0603_1608Metric, symbol Device:R
- added R2, R5, R7: 10K, Resistor_SMD:R_0603_1608Metric, symbol Device:R
- added R3: 1M, Resistor_SMD:R_1206_3216Metric, symbol Device:R
- added R4: 4K7, Resistor_SMD:R_0603_1608Metric, symbol Device:R
- added R6: 200K, Resistor_SMD:R_0603_1608Metric, symbol Device:R
- added SW2: SW_Push, Button_Switch_SMD:SW_SPST_TL3342, symbol Switch:SW_Push
- added U1: AMS1117-5.0, Package_TO_SOT_SMD:SOT-223-3_TabPin2, symbol Regulator_Linear:AMS1117-5.0
- added U15: 74HC14, Package_SO:SOIC-14_3.9x8.7mm_P1.27mm, symbol 74xx:74HC14
- added U2: AMS1117-3.3, Package_TO_SOT_SMD:SOT-223-3_TabPin2, symbol Regulator_Linear:AMS1117-3.3
- added U3: MT3608, Package_TO_SOT_SMD:SOT-23-6, symbol Regulator_Switching:MT3608
- JP1, JP2, JP3, JP4, JP5, JP6, JP7: footprint (none) -> Jumper:SolderJumper-2_P1.3mm_Open_TrianglePad1.0x1.5mm
- U10, U11, U4, U5, U6, U7, U8, U9: footprint (none) -> Package_SO:SOIC-16_3.9x9.9mm_P1.27mm; LCSC (none) -> C5947
- U13: renamed from U3; footprint (none) -> IGG1:IGG1-Anode
- U14: renamed from U2; footprint MCU_RaspberryPi_and_Boards:RP2040-QFN-56 -> Package_DFN_QFN:QFN-56-1EP_7x7mm_P0.4mm_EP3.2x3.2mm
- renumbered C12 to C16, C13 to C17, C14 to C18, C15 to C19, C16 to C20, C17 to C21, C18 to C22, C19 to C23, C20 to C24, C21 to C25, C22 to C26, C23 to C27, C24 to C28, C25 to C29, D18 to D8, J22 to J5, J21 to J6, R51 to R10, R52 to R11, R53 to R12, R54 to R13, R55 to R14, R56 to R15, R49 to R8, R50 to R9, U1 to U12
Connections:
- net +12V: now also C1.1, C2.1, J3.4 (Pin_4), R1.1, U1.3 (VI); no longer D8.1 (K)
- net +3V3: now also C5.1, U2.2 (VO)
- net +5V: now also D8.1 (K), C10.1, C11.1, C12.1, C13.1, C14.1, C3.1, C4.1, C7.1, C8.1, C9.1, D1.3 (VDD), D2.3 (VDD), D3.3 (VDD), D4.3 (VDD), D5.3 (VDD), D6.3 (VDD), J2.1 (Pin_1), U1.2 (VO), U15.14 (VCC), U2.3 (VI)
- net GND: now also C1.2, C10.2, C11.2, C12.2, C13.2, C14.2, C15.2, C2.2, C3.2, C4.2, C5.2, C6.2, C7.2, C8.2, C9.2, D1.1 (VSS), D2.1 (VSS), D3.1 (VSS), D4.1 (VSS), D5.1 (VSS), D6.1 (VSS), J1.2 (Pin_2), J2.5 (Pin_5), J3.1 (Pin_1), J4.2 (Pin_2), R2.1, R4.2, R5.2, R7.2, SW2.1, U1.1 (GND), U15.7 (GND), U2.1 (GND), U3.2 (GND)
- net HV_DIV: now also U14.38 (GPIO26_ADC0), R3.2, R4.1
- net RST: now also SW2.2
- net SR_SHCP: now also U14.11 (GPIO8)
- net SR_STCP: now also U14.17 (GPIO14)
- net ~SR_MC: now also U14.16 (GPIO13)
- net ~SR_OE: now also U14.18 (GPIO15)
- net VUSB: now reaches D8.2 (A), J6.A4 (VBUS), J6.A9 (VBUS), J6.B4 (VBUS), J6.B9 (VBUS)
- net VUSB: now also C6.1, L1.1, U3.5 (IN)
- net K_RST: now reaches U14.14 (GPIO11)
- net K_RST: now also U15.11
- net K_CLK: now reaches U14.15 (GPIO12)
- net K_CLK: now also U15.13
- net K_ADDR_LED: now reaches U14.34 (GPIO22)
- net K_ADDR_LED: now also U15.1
- net A_ADDR_LED: now reaches U14.35 (GPIO23)
- net A_ADDR_LED: now also U15.5
- new net: D4.4 (DOUT), D5.2 (DIN)
- new net: D5.4 (DOUT), D6.2 (DIN)
- new net: D1.4 (DOUT), D2.2 (DIN)
- new net: D7.1 (K), L1.2, U3.1 (SW)
- new net: C15.1, D7.2 (A), R6.1
- new net: R6.2, R7.1, U3.3 (FB)
- new net: D2.4 (DOUT), D3.2 (DIN)
- new net: D3.4 (DOUT), D4.2 (DIN)
- new net: U15.2, U15.3
- new net: U15.6, U15.9
- new net A_ADDR_LED_5V: D1.2 (DIN), U15.8
- new net BAT_DIV: R1.2, R2.2
- new net CHARGE_EN: R5.1, U3.4 (EN)
- new net HT: J1.1 (Pin_1), J4.1 (Pin_1), R3.1
- new net K_ADDR_LED_5V: J2.2 (Pin_2), U15.4
- new net K_CLK_5V: J2.3 (Pin_3), U15.12
- new net K_RST_5V: J2.4 (Pin_4), U15.10
