File: pcb/IGG1_OctoDriver.kicad_pcb (KiCad board)
At the start: 2 copper layers, 50.2 x 25.4 mm, 135 parts, among them J1 Conn_01x01, J10 Conn_01x01, J11 Conn_01x01, J12 Conn_01x01, J13 Conn_01x01, J14 Conn_01x01, J15 Conn_01x01, J16 Conn_01x01, J17 Conn_01x01, J18 Conn_01x01, J19 TEST_1P, J2 Conn_01x08, J3 Conn_01x08, J4 Conn_01x01, J5 Conn_01x08, J6 Conn_01x08, J7 Conn_01x08, J8 Conn_01x08, J9 Conn_01x01, Q1 Q_NPN_BEC, Q10 Q_NPN_BEC, Q11 Q_NPN_BEC, Q12 Q_NPN_BEC, Q13 Q_NPN_BEC, Q14 Q_NPN_BEC, Q15 Q_NPN_BEC, Q16 Q_NPN_BEC, Q17 Q_NPN_BEC, Q18 Q_NPN_BEC, Q19 Q_NPN_BEC, Q2 Q_NPN_BEC, Q20 Q_NPN_BEC, Q21 Q_NPN_BEC, Q22 Q_NPN_BEC, Q23 Q_NPN_BEC, Q24 Q_NPN_BEC, Q3 Q_NPN_BEC, Q4 Q_NPN_BEC, Q5 Q_NPN_BEC, Q6 Q_NPN_BEC, Q7 Q_NPN_BEC, Q8 Q_NPN_BEC, Q9 Q_NPN_BEC, U1 DiodeArray, U10 74LS541, U2 DiodeArray, U3 DiodeArray, U4 DiodeArray, U5 DiodeArray, U6 DiodeArray, U7 DiodeArray, U8 DiodeArray, U9 74LS541

Commit message: Schematic of anode basically done, started layout
Parts:
- removed J10, J11, J12, J13, J14, J15, J16, J17, J18, J9: Conn_01x01, Pin_Headers:Pin_Header_Straight_1x01_Pitch2.54mm
- removed J19 (x21): TEST_1P, footprints:via
- removed J7, J8: Conn_01x08, footprints:Pin_Header_1x08_Pitch1.27mm_SMD
- removed REF** (x4): MountingHole_2.2mm_M2, Mounting_Holes:MountingHole_2.2mm_M2
- added C11: 1u, Capacitor_SMD:C_0603_1608Metric, F.Cu at (212.4, 32.5)
- added C12: 1u, Capacitor_SMD:C_0603_1608Metric, F.Cu at (212.4, 35.0)
- added C13: 1u, Capacitor_SMD:C_0603_1608Metric, F.Cu at (212.4, 37.5)
- added C14: 1u, Capacitor_SMD:C_0603_1608Metric, F.Cu at (212.4, 40.0)
- added C15: 22u, Capacitor_SMD:C_1206_3216Metric, F.Cu at (243.2, 47.0)
- added C16: 100nf, Capacitor_SMD:C_0603_1608Metric, F.Cu at (212.4, 42.5)
- added C17: 4.7pF, Capacitor_SMD:C_0603_1608Metric, F.Cu at (216.5, 27.5)
- added C18: 100nf, Capacitor_SMD:C_0603_1608Metric, F.Cu at (216.5, 30.0)
- added C19: 4.7pF, Capacitor_SMD:C_0603_1608Metric, F.Cu at (216.5, 32.5)
- added C20: 100nf, Capacitor_SMD:C_0603_1608Metric, F.Cu at (216.5, 35.0)
- added C21: 1uf, Capacitor_SMD:C_0603_1608Metric, F.Cu at (216.5, 37.5)
- added C22: 100nf, Capacitor_SMD:C_0603_1608Metric, F.Cu at (216.5, 40.0)
- added C23: 100nf, Capacitor_SMD:C_0603_1608Metric, F.Cu at (216.5, 42.5)
- added C24: 1uf, Capacitor_SMD:C_0603_1608Metric, F.Cu at (220.5, 27.5)
- added C25: 100nf, Capacitor_SMD:C_0603_1608Metric, F.Cu at (220.5, 30.0)
- added C26: 100nf, Capacitor_SMD:C_0603_1608Metric, F.Cu at (220.5, 32.5)
- added C27: 100nf, Capacitor_SMD:C_0603_1608Metric, F.Cu at (220.5, 35.0)
- added C28: 100nf, Capacitor_SMD:C_0603_1608Metric, F.Cu at (220.5, 37.5)
- added C29: 100nf, Capacitor_SMD:C_0603_1608Metric, F.Cu at (220.5, 40.0)
- added C30: 1n, Capacitor_SMD:C_1206_3216Metric, F.Cu at (22.3, -3.00)
- added C31: 1n, Capacitor_SMD:C_1206_3216Metric, F.Cu at (59.5, 101.7)
- added C32: 1n, Capacitor_SMD:C_1206_3216Metric, F.Cu at (42.7, 117.0)
- added C33: 1n, Capacitor_SMD:C_1206_3216Metric, F.Cu at (55.9, 27.4)
- added C34: 1n, Capacitor_SMD:C_1206_3216Metric, F.Cu at (22.3, 42.7)
- added C35: 1n, Capacitor_SMD:C_1206_3216Metric, F.Cu at (-44.8, 27.4)
- added C36: 1n, Capacitor_SMD:C_1206_3216Metric, F.Cu at (-44.8, 42.7)
- added C37: 1n, Capacitor_SMD:C_1206_3216Metric, F.Cu at (-61.6, 12.2)
- added C38: 1n, Capacitor_SMD:C_1206_3216Metric, F.Cu at (5.53, 42.7)
- added C39: 1n, Capacitor_SMD:C_1206_3216Metric, F.Cu at (5.53, 103.5)
- added C40: 1n, Capacitor_SMD:C_1206_3216Metric, F.Cu at (-28.1, 103.5)
- added C41: 1n, Capacitor_SMD:C_1206_3216Metric, F.Cu at (-44.8, 57.9)
- added C42: 1n, Capacitor_SMD:C_1206_3216Metric, F.Cu at (-61.6, 88.3)
- added C43: 1n, Capacitor_SMD:C_1206_3216Metric, F.Cu at (39.1, -3.00)
- added C44: 1n, Capacitor_SMD:C_1206_3216Metric, F.Cu at (-11.3, 103.5)
- added C45: 1n, Capacitor_SMD:C_1206_3216Metric, F.Cu at (-11.3, 27.4)
- added C46: 1n, Capacitor_SMD:C_1206_3216Metric, F.Cu at (22.3, 103.5)
- added C47: 1n, Capacitor_SMD:C_1206_3216Metric, F.Cu at (-11.3, 42.7)
- added C48: 1n, Capacitor_SMD:C_1206_3216Metric, F.Cu at (-11.3, -3.00)
- added C49: 1n, Capacitor_SMD:C_1206_3216Metric, F.Cu at (-28.1, -3.00)
- added C50: 1n, Capacitor_SMD:C_1206_3216Metric, F.Cu at (55.9, 12.2)
- added C51: 1n, Capacitor_SMD:C_1206_3216Metric, F.Cu at (-44.8, 88.3)
- added C52: 1n, Capacitor_SMD:C_1206_3216Metric, F.Cu at (39.1, 88.3)
- added C53: 1n, Capacitor_SMD:C_1206_3216Metric, F.Cu at (55.9, -3.00)
- added C54: 1n, Capacitor_SMD:C_1206_3216Metric, F.Cu at (-11.3, 73.1)
- added C55: 1n, Capacitor_SMD:C_1206_3216Metric, F.Cu at (165.5, 131.0)
- added C56: 1n, Capacitor_SMD:C_1206_3216Metric, F.Cu at (-11.3, 57.9)
- added C57: 1n, Capacitor_SMD:C_1206_3216Metric, F.Cu at (39.1, 27.4)
- added C58: 1n, Capacitor_SMD:C_1206_3216Metric, F.Cu at (-61.6, 57.9)
- added C59: 1n, Capacitor_SMD:C_1206_3216Metric, F.Cu at (5.53, 73.1)
- added C60: 1n, Capacitor_SMD:C_1206_3216Metric, F.Cu at (55.9, 42.7)
- added C61: 1n, Capacitor_SMD:C_1206_3216Metric, F.Cu at (22.3, 57.9)
- added C62: 1n, Capacitor_SMD:C_1206_3216Metric, F.Cu at (39.1, 57.9)
- added C63: 1n, Capacitor_SMD:C_1206_3216Metric, F.Cu at (55.9, 57.9)
- added C64: 1n, Capacitor_SMD:C_1206_3216Metric, F.Cu at (-61.6, 73.1)
- added C65: 1n, Capacitor_SMD:C_1206_3216Metric, F.Cu at (-28.1, 73.1)
- added C66: 1n, Capacitor_SMD:C_1206_3216Metric, F.Cu at (-61.6, 42.7)
- added C67: 1n, Capacitor_SMD:C_1206_3216Metric, F.Cu at (-28.1, 42.7)
- added C68: 1n, Capacitor_SMD:C_1206_3216Metric, F.Cu at (39.1, 42.7)
- added C69: 1n, Capacitor_SMD:C_1206_3216Metric, F.Cu at (-61.6, 27.4)
- added C70: 1n, Capacitor_SMD:C_1206_3216Metric, F.Cu at (-61.6, -3.00)
- added C71: 1n, Capacitor_SMD:C_1206_3216Metric, F.Cu at (-28.1, 57.9)
- added C72: 1n, Capacitor_SMD:C_1206_3216Metric, F.Cu at (-44.8, 12.2)
- added C73: 1n, Capacitor_SMD:C_1206_3216Metric, F.Cu at (5.53, 88.3)
- added C74: 1n, Capacitor_SMD:C_1206_3216Metric, F.Cu at (5.53, 12.2)
- added C75: 1n, Capacitor_SMD:C_1206_3216Metric, F.Cu at (5.53, 57.9)
- added C76: 1n, Capacitor_SMD:C_1206_3216Metric, F.Cu at (-44.8, 73.1)
- added C77: 1n, Capacitor_SMD:C_1206_3216Metric, F.Cu at (-61.6, 103.5)
- added C78: 1n, Capacitor_SMD:C_1206_3216Metric, F.Cu at (5.53, -3.00)
- added C79: 1n, Capacitor_SMD:C_1206_3216Metric, F.Cu at (22.3, 73.1)
- added C80: 1n, Capacitor_SMD:C_1206_3216Metric, F.Cu at (-28.1, 12.2)
- added C81: 1n, Capacitor_SMD:C_1206_3216Metric, F.Cu at (22.3, 12.2)
- added C82: 1n, Capacitor_SMD:C_1206_3216Metric, F.Cu at (-11.3, 12.2)
- added C83: 1n, Capacitor_SMD:C_1206_3216Metric, F.Cu at (-44.8, 103.5)
- added C84: 1n, Capacitor_SMD:C_1206_3216Metric, F.Cu at (22.3, 27.4)
- added C85: 1n, Capacitor_SMD:C_1206_3216Metric, F.Cu at (-28.1, 27.4)
- added C86: 1n, Capacitor_SMD:C_1206_3216Metric, F.Cu at (39.1, 73.1)
- added C87: 1n, Capacitor_SMD:C_1206_3216Metric, F.Cu at (-44.8, -3.00)
- added C88: 1n, Capacitor_SMD:C_1206_3216Metric, F.Cu at (-28.1, 88.3)
- added C89: 1n, Capacitor_SMD:C_1206_3216Metric, F.Cu at (5.53, 27.4)
- added C90: 1n, Capacitor_SMD:C_1206_3216Metric, F.Cu at (39.1, 12.2)
- added C91: 1n, Capacitor_SMD:C_1206_3216Metric, F.Cu at (22.3, 88.3)
- added C92: 1n, Capacitor_SMD:C_1206_3216Metric, F.Cu at (-11.3, 88.3)
- added C93: 1n, Capacitor_SMD:C_1206_3216Metric, F.Cu at (271.0, 84.5)
- added D1: SK6812, LED_SMD:LED_SK6812MINI_PLCC4_3.5x3.5mm_P1.75mm, F.Cu at (195.8, 28.7)
- added D10: D, Diode_SMD:D_SOD-323, F.Cu at (19.3, -3.46)
- added D100: D, Diode_SMD:D_SOD-323, F.Cu at (2.52, 57.4)
- added D101: D, Diode_SMD:D_SOD-323, F.Cu at (-43.3, 81.6)
- added D102: D, Diode_SMD:D_SOD-323, F.Cu at (-47.8, 72.6)
- added D103: D, Diode_SMD:D_SOD-323, F.Cu at (-60.1, 112.0)
- added D104: D, Diode_SMD:D_SOD-323, F.Cu at (-64.6, 103.1)
- added D105: D, Diode_SMD:D_SOD-323, F.Cu at (7.03, 5.50)
- added D106: D, Diode_SMD:D_SOD-323, F.Cu at (2.52, -3.46)
- added D107: D, Diode_SMD:D_SOD-323, F.Cu at (23.8, 81.6)
- added D108: D, Diode_SMD:D_SOD-323, F.Cu at (19.3, 72.6)
- added D109: D, Diode_SMD:D_SOD-323, F.Cu at (-26.6, 20.7)
- added D11: D, Diode_SMD:D_SOD-323, F.Cu at (229.8, 75.8)
- added D110: D, Diode_SMD:D_SOD-323, F.Cu at (-31.1, 11.8)
- added D111: D, Diode_SMD:D_SOD-323, F.Cu at (23.8, 20.7)
- added D112: D, Diode_SMD:D_SOD-323, F.Cu at (19.3, 11.8)
- added D113: D, Diode_SMD:D_SOD-323, F.Cu at (-9.77, 20.7)
- added D114: D, Diode_SMD:D_SOD-323, F.Cu at (-14.3, 11.8)
- added D115: D, Diode_SMD:D_SOD-323, F.Cu at (-43.3, 112.0)
- added D116: D, Diode_SMD:D_SOD-323, F.Cu at (-47.8, 103.1)
- added D117: D, Diode_SMD:D_SOD-323, F.Cu at (23.8, 35.9)
- added D118: D, Diode_SMD:D_SOD-323, F.Cu at (19.3, 27.0)
- added D119: D, Diode_SMD:D_SOD-323, F.Cu at (-26.6, 35.9)
- added D12: D, Diode_SMD:D_SOD-323, F.Cu at (229.8, 78.7)
- added D120: D, Diode_SMD:D_SOD-323, F.Cu at (-31.1, 27.0)
- added D121: D, Diode_SMD:D_SOD-323, F.Cu at (40.6, 81.6)
- added D122: D, Diode_SMD:D_SOD-323, F.Cu at (36.1, 72.6)
- added D123: D, Diode_SMD:D_SOD-323, F.Cu at (-43.3, 5.50)
- added D124: D, Diode_SMD:D_SOD-323, F.Cu at (-47.8, -3.46)
- added D125: D, Diode_SMD:D_SOD-323, F.Cu at (-26.6, 96.8)
- added D126: D, Diode_SMD:D_SOD-323, F.Cu at (-31.1, 87.9)
- added D127: D, Diode_SMD:D_SOD-323, F.Cu at (7.03, 35.9)
- added D128: D, Diode_SMD:D_SOD-323, F.Cu at (2.52, 27.0)
- added D129: D, Diode_SMD:D_SOD-323, F.Cu at (40.6, 20.7)
- added D13: D, Diode_SMD:D_SOD-323, F.Cu at (168.0, 75.8)
- added D130: D, Diode_SMD:D_SOD-323, F.Cu at (36.1, 11.8)
- added D131: D, Diode_SMD:D_SOD-323, F.Cu at (23.8, 96.8)
- added D132: D, Diode_SMD:D_SOD-323, F.Cu at (19.3, 87.9)
- added D133: D, Diode_SMD:D_SOD-323, F.Cu at (-9.77, 96.8)
- added D134: D, Diode_SMD:D_SOD-323, F.Cu at (-14.3, 87.9)
- added D135: D, Diode_SMD:D_SOD-323, F.Cu at (272.5, 93.0)
- added D136: D, Diode_SMD:D_SOD-323, F.Cu at (268.0, 84.0)
- added D14: D, Diode_SMD:D_SOD-323, F.Cu at (168.0, 78.7)
- added D15: D, Diode_SMD:D_SOD-323, F.Cu at (57.4, 35.9)
- added D16: D, Diode_SMD:D_SOD-323, F.Cu at (52.9, 27.0)
- added D17: D, Diode_SMD:D_SOD-323, F.Cu at (23.8, 51.2)
- added D18: D, Diode_SMD:D_SOD-323, F.Cu at (19.3, 42.2)
- added D19: D, Diode_SMD:D_SOD-323, F.Cu at (-43.3, 35.9)
- added D2: SK6812, LED_SMD:LED_SK6812MINI_PLCC4_3.5x3.5mm_P1.75mm, F.Cu at (195.8, 33.8)
- added D20: D, Diode_SMD:D_SOD-323, F.Cu at (-47.8, 27.0)
- added D21: D, Diode_SMD:D_SOD-323, F.Cu at (-43.3, 51.2)
- added D22: D, Diode_SMD:D_SOD-323, F.Cu at (-47.8, 42.2)
- added D23: D, Diode_SMD:D_SOD-323, F.Cu at (-60.1, 20.7)
- added D24: D, Diode_SMD:D_SOD-323, F.Cu at (-64.6, 11.8)
- added D25: D, Diode_SMD:D_SOD-323, F.Cu at (7.03, 51.2)
- added D26: D, Diode_SMD:D_SOD-323, F.Cu at (2.52, 42.2)
- added D27: D, Diode_SMD:D_SOD-323, F.Cu at (7.03, 112.0)
- added D28: D, Diode_SMD:D_SOD-323, F.Cu at (2.52, 103.1)
- added D29: D, Diode_SMD:D_SOD-323, F.Cu at (-26.6, 112.0)
- added D3: SK6812, LED_SMD:LED_SK6812MINI_PLCC4_3.5x3.5mm_P1.75mm, F.Cu at (195.8, 38.8)
- added D30: D, Diode_SMD:D_SOD-323, F.Cu at (-31.1, 103.1)
- added D31: D, Diode_SMD:D_SOD-323, F.Cu at (-43.3, 66.4)
- added D32: D, Diode_SMD:D_SOD-323, F.Cu at (-47.8, 57.4)
- added D33: D, Diode_SMD:D_SOD-323, F.Cu at (-60.1, 96.8)
- added D34: D, Diode_SMD:D_SOD-323, F.Cu at (-64.6, 87.9)
- added D35: D, Diode_SMD:D_SOD-323, F.Cu at (40.6, 5.50)
- added D36: D, Diode_SMD:D_SOD-323, F.Cu at (36.1, -3.46)
- added D37: D, Diode_SMD:D_SOD-323, F.Cu at (-9.77, 112.0)
- added D38: D, Diode_SMD:D_SOD-323, F.Cu at (-14.3, 103.1)
- added D39: D, Diode_SMD:D_SOD-323, F.Cu at (-9.77, 35.9)
- added D4: SK6812, LED_SMD:LED_SK6812MINI_PLCC4_3.5x3.5mm_P1.75mm, F.Cu at (195.8, 43.9)
- added D40: D, Diode_SMD:D_SOD-323, F.Cu at (-14.3, 27.0)
- added D41: D, Diode_SMD:D_SOD-323, F.Cu at (23.8, 112.0)
- added D42: D, Diode_SMD:D_SOD-323, F.Cu at (19.3, 103.1)
- added D43: D, Diode_SMD:D_SOD-323, F.Cu at (-9.77, 51.2)
- added D44: D, Diode_SMD:D_SOD-323, F.Cu at (-14.3, 42.2)
- added D45: D, Diode_SMD:D_SOD-323, F.Cu at (-9.77, 5.50)
- added D46: D, Diode_SMD:D_SOD-323, F.Cu at (-14.3, -3.46)
- added D47: D, Diode_SMD:D_SOD-323, F.Cu at (-26.6, 5.50)
- added D48: D, Diode_SMD:D_SOD-323, F.Cu at (-31.1, -3.46)
- added D49: D, Diode_SMD:D_SOD-323, F.Cu at (57.4, 20.7)
- added D5: SK6812, LED_SMD:LED_SK6812MINI_PLCC4_3.5x3.5mm_P1.75mm, F.Cu at (195.8, 48.9)
- added D50: D, Diode_SMD:D_SOD-323, F.Cu at (52.9, 11.8)
- added D51: D, Diode_SMD:D_SOD-323, F.Cu at (-43.3, 96.8)
- added D52: D, Diode_SMD:D_SOD-323, F.Cu at (-47.8, 87.9)
- added D53: D, Diode_SMD:D_SOD-323, F.Cu at (40.6, 96.8)
- added D54: D, Diode_SMD:D_SOD-323, F.Cu at (36.1, 87.9)
- added D55: D, Diode_SMD:D_SOD-323, F.Cu at (57.4, 5.50)
- added D56: D, Diode_SMD:D_SOD-323, F.Cu at (52.9, -3.46)
- added D57: D, Diode_SMD:D_SOD-323, F.Cu at (-9.77, 81.6)
- added D58: D, Diode_SMD:D_SOD-323, F.Cu at (-14.3, 72.6)
- added D59: D, Diode_SMD:D_SOD-323, F.Cu at (167.0, 139.5)
- added D6: SK6812, LED_SMD:LED_SK6812MINI_PLCC4_3.5x3.5mm_P1.75mm, F.Cu at (195.8, 54.0)
- added D60: D, Diode_SMD:D_SOD-323, F.Cu at (162.5, 130.6)
- added D61: D, Diode_SMD:D_SOD-323, F.Cu at (-9.77, 66.4)
- added D62: D, Diode_SMD:D_SOD-323, F.Cu at (-14.3, 57.4)
- added D63: D, Diode_SMD:D_SOD-323, F.Cu at (40.6, 35.9)
- added D64: D, Diode_SMD:D_SOD-323, F.Cu at (36.1, 27.0)
- added D65: D, Diode_SMD:D_SOD-323, F.Cu at (-60.1, 66.4)
- added D66: D, Diode_SMD:D_SOD-323, F.Cu at (-64.6, 57.4)
- added D67: D, Diode_SMD:D_SOD-323, F.Cu at (7.03, 81.6)
- added D68: D, Diode_SMD:D_SOD-323, F.Cu at (2.52, 72.6)
- added D69: D, Diode_SMD:D_SOD-323, F.Cu at (57.4, 51.2)
- added D7: D, Diode_SMD:D_SMA, F.Cu at (268.4, 45.7)
- added D70: D, Diode_SMD:D_SOD-323, F.Cu at (52.9, 42.2)
- added D71: D, Diode_SMD:D_SOD-323, F.Cu at (23.8, 66.4)
- added D72: D, Diode_SMD:D_SOD-323, F.Cu at (19.3, 57.4)
- added D73: D, Diode_SMD:D_SOD-323, F.Cu at (40.6, 66.4)
- added D74: D, Diode_SMD:D_SOD-323, F.Cu at (36.1, 57.4)
- added D75: D, Diode_SMD:D_SOD-323, F.Cu at (57.4, 66.4)
- added D76: D, Diode_SMD:D_SOD-323, F.Cu at (52.9, 57.4)
- added D77: D, Diode_SMD:D_SOD-323, F.Cu at (-60.1, 81.6)
- added D78: D, Diode_SMD:D_SOD-323, F.Cu at (-64.6, 72.6)
- added D79: D, Diode_SMD:D_SOD-323, F.Cu at (-26.6, 81.6)
- added D8: D, Diode_SMD:D_SMA, F.Cu at (268.4, 50.3)
- added D80: D, Diode_SMD:D_SOD-323, F.Cu at (-31.1, 72.6)
- added D81: D, Diode_SMD:D_SOD-323, F.Cu at (-60.1, 51.2)
- added D82: D, Diode_SMD:D_SOD-323, F.Cu at (-64.6, 42.2)
- added D83: D, Diode_SMD:D_SOD-323, F.Cu at (-26.6, 51.2)
- added D84: D, Diode_SMD:D_SOD-323, F.Cu at (-31.1, 42.2)
- added D85: D, Diode_SMD:D_SOD-323, F.Cu at (40.6, 51.2)
- added D86: D, Diode_SMD:D_SOD-323, F.Cu at (36.1, 42.2)
- added D87: D, Diode_SMD:D_SOD-323, F.Cu at (-60.1, 35.9)
- added D88: D, Diode_SMD:D_SOD-323, F.Cu at (-64.6, 27.0)
- added D89: D, Diode_SMD:D_SOD-323, F.Cu at (-60.1, 5.50)
- added D9: D, Diode_SMD:D_SOD-323, F.Cu at (23.8, 5.50)
- added D90: D, Diode_SMD:D_SOD-323, F.Cu at (-64.6, -3.46)
- added D91: D, Diode_SMD:D_SOD-323, F.Cu at (-26.6, 66.4)
- added D92: D, Diode_SMD:D_SOD-323, F.Cu at (-31.1, 57.4)
- added D93: D, Diode_SMD:D_SOD-323, F.Cu at (-43.3, 20.7)
- added D94: D, Diode_SMD:D_SOD-323, F.Cu at (-47.8, 11.8)
- added D95: D, Diode_SMD:D_SOD-323, F.Cu at (7.03, 96.8)
- added D96: D, Diode_SMD:D_SOD-323, F.Cu at (2.52, 87.9)
- added D97: D, Diode_SMD:D_SOD-323, F.Cu at (7.03, 20.7)
- added D98: D, Diode_SMD:D_SOD-323, F.Cu at (2.52, 11.8)
- added D99: D, Diode_SMD:D_SOD-323, F.Cu at (7.03, 66.4)
- added H1: H, MountingHole:MountingHole_3.2mm_M3_DIN965_Pad, F.Cu at (202.9, 29.8)
- added H2: H, MountingHole:MountingHole_3.2mm_M3_DIN965_Pad, F.Cu at (202.9, 36.9)
- added H3: H, MountingHole:MountingHole_3.2mm_M3_DIN965_Pad, F.Cu at (202.9, 44.1)
- added H4: H, MountingHole:MountingHole_3.2mm_M3_DIN965_Pad, F.Cu at (202.9, 51.2)
- added JP1: Jumper_2_Open, Jumper:SolderJumper-2_P1.3mm_Open_TrianglePad1.0x1.5mm, F.Cu at (90.7, 93.9)
- added JP2: Jumper_2_Open, Jumper:SolderJumper-2_P1.3mm_Open_TrianglePad1.0x1.5mm, F.Cu at (90.7, 97.5)
- added JP3: Jumper_2_Open, Jumper:SolderJumper-2_P1.3mm_Open_TrianglePad1.0x1.5mm, F.Cu at (90.7, 101.0)
- added JP4: Jumper_2_Open, Jumper:SolderJumper-2_P1.3mm_Open_TrianglePad1.0x1.5mm, F.Cu at (90.7, 104.6)
- added JP5: Jumper_2_Open, Jumper:SolderJumper-2_P1.3mm_Open_TrianglePad1.0x1.5mm, F.Cu at (90.7, 108.1)
- added JP6: Jumper_2_Open, Jumper:SolderJumper-2_P1.3mm_Open_TrianglePad1.0x1.5mm, F.Cu at (90.7, 111.7)
- added JP7: Jumper_2_Open, Jumper:SolderJumper-2_P1.3mm_Open_TrianglePad1.0x1.5mm, F.Cu at (90.7, 115.2)
- added L1: 22uH, Inductor_SMD:L_Chilisin_BMRF00101040, F.Cu at (257.1, 32.1)
- added Q100: Q_NPN_BEC, Package_TO_SOT_SMD:SOT-23, F.Cu at (21.8, 84.1)
- added Q101: Q_NPN_BEC, Package_TO_SOT_SMD:SOT-23, F.Cu at (-27.6, 16.7)
- added Q102: Q_NPN_BEC, Package_TO_SOT_SMD:SOT-23, F.Cu at (-28.6, 23.2)
- added Q103: Q_NPN_BEC, Package_TO_SOT_SMD:SOT-23, F.Cu at (22.8, 16.7)
- added Q104: Q_NPN_BEC, Package_TO_SOT_SMD:SOT-23, F.Cu at (21.8, 23.2)
- added Q105: Q_NPN_BEC, Package_TO_SOT_SMD:SOT-23, F.Cu at (-10.8, 16.7)
- added Q106: Q_NPN_BEC, Package_TO_SOT_SMD:SOT-23, F.Cu at (-11.8, 23.2)
- added Q107: Q_NPN_BEC, Package_TO_SOT_SMD:SOT-23, F.Cu at (-44.3, 108.0)
- added Q108: Q_NPN_BEC, Package_TO_SOT_SMD:SOT-23, F.Cu at (-45.3, 114.5)
- added Q109: Q_NPN_BEC, Package_TO_SOT_SMD:SOT-23, F.Cu at (22.8, 31.9)
- added Q110: Q_NPN_BEC, Package_TO_SOT_SMD:SOT-23, F.Cu at (21.8, 38.4)
- added Q111: Q_NPN_BEC, Package_TO_SOT_SMD:SOT-23, F.Cu at (-27.6, 31.9)
- added Q112: Q_NPN_BEC, Package_TO_SOT_SMD:SOT-23, F.Cu at (-28.6, 38.4)
- added Q113: Q_NPN_BEC, Package_TO_SOT_SMD:SOT-23, F.Cu at (39.6, 77.6)
- added Q114: Q_NPN_BEC, Package_TO_SOT_SMD:SOT-23, F.Cu at (38.6, 84.1)
- added Q115: Q_NPN_BEC, Package_TO_SOT_SMD:SOT-23, F.Cu at (-44.3, 1.50)
- added Q116: Q_NPN_BEC, Package_TO_SOT_SMD:SOT-23, F.Cu at (-45.3, 8.00)
- added Q117: Q_NPN_BEC, Package_TO_SOT_SMD:SOT-23, F.Cu at (-27.6, 92.8)
- added Q118: Q_NPN_BEC, Package_TO_SOT_SMD:SOT-23, F.Cu at (-28.6, 99.3)
- added Q119: Q_NPN_BEC, Package_TO_SOT_SMD:SOT-23, F.Cu at (6.03, 31.9)
- added Q120: Q_NPN_BEC, Package_TO_SOT_SMD:SOT-23, F.Cu at (5.03, 38.4)
- added Q121: Q_NPN_BEC, Package_TO_SOT_SMD:SOT-23, F.Cu at (39.6, 16.7)
- added Q122: Q_NPN_BEC, Package_TO_SOT_SMD:SOT-23, F.Cu at (38.6, 23.2)
- added Q123: Q_NPN_BEC, Package_TO_SOT_SMD:SOT-23, F.Cu at (22.8, 92.8)
- added Q124: Q_NPN_BEC, Package_TO_SOT_SMD:SOT-23, F.Cu at (21.8, 99.3)
- added Q125: Q_NPN_BEC, Package_TO_SOT_SMD:SOT-23, F.Cu at (-10.8, 92.8)
- added Q126: Q_NPN_BEC, Package_TO_SOT_SMD:SOT-23, F.Cu at (-11.8, 99.3)
- added Q127: Q_NPN_BEC, Package_TO_SOT_SMD:SOT-23, F.Cu at (271.5, 89.0)
- added Q128: Q_NPN_BEC, Package_TO_SOT_SMD:SOT-23, F.Cu at (270.5, 95.5)
- added Q25: Q_NPN_BEC, Package_TO_SOT_SMD:SOT-23, F.Cu at (-61.1, 92.8)
- added Q26: Q_NPN_BEC, Package_TO_SOT_SMD:SOT-23, F.Cu at (-62.1, 99.3)
- added Q27: Q_NPN_BEC, Package_TO_SOT_SMD:SOT-23, F.Cu at (39.6, 1.50)
- added Q28: Q_NPN_BEC, Package_TO_SOT_SMD:SOT-23, F.Cu at (38.6, 8.00)
- added Q29: Q_NPN_BEC, Package_TO_SOT_SMD:SOT-23, F.Cu at (-10.8, 108.0)
- added Q30: Q_NPN_BEC, Package_TO_SOT_SMD:SOT-23, F.Cu at (-11.8, 114.5)
- added Q31: Q_NPN_BEC, Package_TO_SOT_SMD:SOT-23, F.Cu at (-10.8, 31.9)
- added Q32: Q_NPN_BEC, Package_TO_SOT_SMD:SOT-23, F.Cu at (-11.8, 38.4)
- added Q33: Q_NPN_BEC, Package_TO_SOT_SMD:SOT-23, F.Cu at (22.8, 108.0)
- added Q34: Q_NPN_BEC, Package_TO_SOT_SMD:SOT-23, F.Cu at (21.8, 114.5)
- added Q35: Q_NPN_BEC, Package_TO_SOT_SMD:SOT-23, F.Cu at (-10.8, 47.2)
- added Q36: Q_NPN_BEC, Package_TO_SOT_SMD:SOT-23, F.Cu at (-11.8, 53.7)
- added Q37: Q_NPN_BEC, Package_TO_SOT_SMD:SOT-23, F.Cu at (-10.8, 1.50)
- added Q38: Q_NPN_BEC, Package_TO_SOT_SMD:SOT-23, F.Cu at (-11.8, 8.00)
- added Q39: Q_NPN_BEC, Package_TO_SOT_SMD:SOT-23, F.Cu at (-27.6, 1.50)
- added Q40: Q_NPN_BEC, Package_TO_SOT_SMD:SOT-23, F.Cu at (-28.6, 8.00)
- added Q41: Q_NPN_BEC, Package_TO_SOT_SMD:SOT-23, F.Cu at (56.4, 16.7)
- added Q42: Q_NPN_BEC, Package_TO_SOT_SMD:SOT-23, F.Cu at (55.4, 23.2)
- added Q43: Q_NPN_BEC, Package_TO_SOT_SMD:SOT-23, F.Cu at (-44.3, 92.8)
- added Q44: Q_NPN_BEC, Package_TO_SOT_SMD:SOT-23, F.Cu at (-45.3, 99.3)
- added Q45: Q_NPN_BEC, Package_TO_SOT_SMD:SOT-23, F.Cu at (39.6, 92.8)
- added Q46: Q_NPN_BEC, Package_TO_SOT_SMD:SOT-23, F.Cu at (38.6, 99.3)
- added Q47: Q_NPN_BEC, Package_TO_SOT_SMD:SOT-23, F.Cu at (56.4, 1.50)
- added Q48: Q_NPN_BEC, Package_TO_SOT_SMD:SOT-23, F.Cu at (55.4, 8.00)
- added Q49: Q_NPN_BEC, Package_TO_SOT_SMD:SOT-23, F.Cu at (-10.8, 77.6)
- added Q50: Q_NPN_BEC, Package_TO_SOT_SMD:SOT-23, F.Cu at (-11.8, 84.1)
- added Q51: Q_NPN_BEC, Package_TO_SOT_SMD:SOT-23, F.Cu at (166.0, 135.5)
- added Q52: Q_NPN_BEC, Package_TO_SOT_SMD:SOT-23, F.Cu at (165.0, 142.0)
- added Q53: Q_NPN_BEC, Package_TO_SOT_SMD:SOT-23, F.Cu at (-10.8, 62.4)
- added Q54: Q_NPN_BEC, Package_TO_SOT_SMD:SOT-23, F.Cu at (-11.8, 68.9)
- added Q55: Q_NPN_BEC, Package_TO_SOT_SMD:SOT-23, F.Cu at (39.6, 31.9)
- added Q56: Q_NPN_BEC, Package_TO_SOT_SMD:SOT-23, F.Cu at (38.6, 38.4)
- added Q57: Q_NPN_BEC, Package_TO_SOT_SMD:SOT-23, F.Cu at (-61.1, 62.4)
- added Q58: Q_NPN_BEC, Package_TO_SOT_SMD:SOT-23, F.Cu at (-62.1, 68.9)
- added Q59: Q_NPN_BEC, Package_TO_SOT_SMD:SOT-23, F.Cu at (6.03, 77.6)
- added Q60: Q_NPN_BEC, Package_TO_SOT_SMD:SOT-23, F.Cu at (5.03, 84.1)
- added Q61: Q_NPN_BEC, Package_TO_SOT_SMD:SOT-23, F.Cu at (56.4, 47.2)
- added Q62: Q_NPN_BEC, Package_TO_SOT_SMD:SOT-23, F.Cu at (55.4, 53.7)
- added Q63: Q_NPN_BEC, Package_TO_SOT_SMD:SOT-23, F.Cu at (22.8, 62.4)
- added Q64: Q_NPN_BEC, Package_TO_SOT_SMD:SOT-23, F.Cu at (21.8, 68.9)
- added Q65: Q_NPN_BEC, Package_TO_SOT_SMD:SOT-23, F.Cu at (39.6, 62.4)
- added Q66: Q_NPN_BEC, Package_TO_SOT_SMD:SOT-23, F.Cu at (38.6, 68.9)
- added Q67: Q_NPN_BEC, Package_TO_SOT_SMD:SOT-23, F.Cu at (56.4, 62.4)
- added Q68: Q_NPN_BEC, Package_TO_SOT_SMD:SOT-23, F.Cu at (55.4, 68.9)
- added Q69: Q_NPN_BEC, Package_TO_SOT_SMD:SOT-23, F.Cu at (-61.1, 77.6)
- added Q70: Q_NPN_BEC, Package_TO_SOT_SMD:SOT-23, F.Cu at (-62.1, 84.1)
- added Q71: Q_NPN_BEC, Package_TO_SOT_SMD:SOT-23, F.Cu at (-27.6, 77.6)
- added Q72: Q_NPN_BEC, Package_TO_SOT_SMD:SOT-23, F.Cu at (-28.6, 84.1)
- added Q73: Q_NPN_BEC, Package_TO_SOT_SMD:SOT-23, F.Cu at (-61.1, 47.2)
- added Q74: Q_NPN_BEC, Package_TO_SOT_SMD:SOT-23, F.Cu at (-62.1, 53.7)
- added Q75: Q_NPN_BEC, Package_TO_SOT_SMD:SOT-23, F.Cu at (-27.6, 47.2)
- added Q76: Q_NPN_BEC, Package_TO_SOT_SMD:SOT-23, F.Cu at (-28.6, 53.7)
- added Q77: Q_NPN_BEC, Package_TO_SOT_SMD:SOT-23, F.Cu at (39.6, 47.2)
- added Q78: Q_NPN_BEC, Package_TO_SOT_SMD:SOT-23, F.Cu at (38.6, 53.7)
- added Q79: Q_NPN_BEC, Package_TO_SOT_SMD:SOT-23, F.Cu at (-61.1, 31.9)
- added Q80: Q_NPN_BEC, Package_TO_SOT_SMD:SOT-23, F.Cu at (-62.1, 38.4)
- added Q81: Q_NPN_BEC, Package_TO_SOT_SMD:SOT-23, F.Cu at (-61.1, 1.50)
- added Q82: Q_NPN_BEC, Package_TO_SOT_SMD:SOT-23, F.Cu at (-62.1, 8.00)
- added Q83: Q_NPN_BEC, Package_TO_SOT_SMD:SOT-23, F.Cu at (-27.6, 62.4)
- added Q84: Q_NPN_BEC, Package_TO_SOT_SMD:SOT-23, F.Cu at (-28.6, 68.9)
- added Q85: Q_NPN_BEC, Package_TO_SOT_SMD:SOT-23, F.Cu at (-44.3, 16.7)
- added Q86: Q_NPN_BEC, Package_TO_SOT_SMD:SOT-23, F.Cu at (-45.3, 23.2)
- added Q87: Q_NPN_BEC, Package_TO_SOT_SMD:SOT-23, F.Cu at (6.03, 92.8)
- added Q88: Q_NPN_BEC, Package_TO_SOT_SMD:SOT-23, F.Cu at (5.03, 99.3)
- added Q89: Q_NPN_BEC, Package_TO_SOT_SMD:SOT-23, F.Cu at (6.03, 16.7)
- added Q90: Q_NPN_BEC, Package_TO_SOT_SMD:SOT-23, F.Cu at (5.03, 23.2)
- added Q91: Q_NPN_BEC, Package_TO_SOT_SMD:SOT-23, F.Cu at (6.03, 62.4)
- added Q92: Q_NPN_BEC, Package_TO_SOT_SMD:SOT-23, F.Cu at (5.03, 68.9)
- added Q93: Q_NPN_BEC, Package_TO_SOT_SMD:SOT-23, F.Cu at (-44.3, 77.6)
- added Q94: Q_NPN_BEC, Package_TO_SOT_SMD:SOT-23, F.Cu at (-45.3, 84.1)
- added Q95: Q_NPN_BEC, Package_TO_SOT_SMD:SOT-23, F.Cu at (-61.1, 108.0)
- added Q96: Q_NPN_BEC, Package_TO_SOT_SMD:SOT-23, F.Cu at (-62.1, 114.5)
- added Q97: Q_NPN_BEC, Package_TO_SOT_SMD:SOT-23, F.Cu at (6.03, 1.50)
- added Q98: Q_NPN_BEC, Package_TO_SOT_SMD:SOT-23, F.Cu at (5.03, 8.00)
- added Q99: Q_NPN_BEC, Package_TO_SOT_SMD:SOT-23, F.Cu at (22.8, 77.6)
- added R100: 10K, Resistor_SMD:R_0603_1608Metric, F.Cu at (-48.3, 99.8)
- added R101: 220K, Resistor_SMD:R_1206_3216Metric, F.Cu at (-46.8, 95.8)
- added R102: 100K, Resistor_SMD:R_1206_3216Metric, F.Cu at (-46.3, 83.3)
- added R103: 4.7K, Resistor_SMD:R_1206_3216Metric, F.Cu at (-47.8, 91.9)
- added R104: 10K, Resistor_SMD:R_0603_1608Metric, F.Cu at (35.6, 99.8)
- added R105: 220K, Resistor_SMD:R_1206_3216Metric, F.Cu at (37.1, 95.8)
- added R106: 100K, Resistor_SMD:R_1206_3216Metric, F.Cu at (37.6, 83.3)
- added R107: 4.7K, Resistor_SMD:R_1206_3216Metric, F.Cu at (36.1, 91.9)
- added R108: 10K, Resistor_SMD:R_0603_1608Metric, F.Cu at (52.4, 8.49)
- added R109: 220K, Resistor_SMD:R_1206_3216Metric, F.Cu at (53.9, 4.50)
- added R110: 100K, Resistor_SMD:R_1206_3216Metric, F.Cu at (54.4, -8.01)
- added R111: 4.7K, Resistor_SMD:R_1206_3216Metric, F.Cu at (52.9, 0.55)
- added R112: 10K, Resistor_SMD:R_0603_1608Metric, F.Cu at (-14.8, 84.6)
- added R113: 220K, Resistor_SMD:R_1206_3216Metric, F.Cu at (-13.3, 80.6)
- added R114: 100K, Resistor_SMD:R_1206_3216Metric, F.Cu at (-12.8, 68.1)
- added R115: 4.7K, Resistor_SMD:R_1206_3216Metric, F.Cu at (-14.3, 76.6)
- added R116: 10K, Resistor_SMD:R_0603_1608Metric, F.Cu at (162.0, 142.5)
- added R117: 220K, Resistor_SMD:R_1206_3216Metric, F.Cu at (163.5, 138.5)
- added R118: 100K, Resistor_SMD:R_1206_3216Metric, F.Cu at (164.0, 126.0)
- added R119: 4.7K, Resistor_SMD:R_1206_3216Metric, F.Cu at (162.5, 134.6)
- added R120: 10K, Resistor_SMD:R_0603_1608Metric, F.Cu at (-14.8, 69.4)
- added R121: 220K, Resistor_SMD:R_1206_3216Metric, F.Cu at (-13.3, 65.4)
- added R122: 100K, Resistor_SMD:R_1206_3216Metric, F.Cu at (-12.8, 52.9)
- added R123: 4.7K, Resistor_SMD:R_1206_3216Metric, F.Cu at (-14.3, 61.4)
- added R124: 10K, Resistor_SMD:R_0603_1608Metric, F.Cu at (35.6, 38.9)
- added R125: 220K, Resistor_SMD:R_1206_3216Metric, F.Cu at (37.1, 34.9)
- added R126: 100K, Resistor_SMD:R_1206_3216Metric, F.Cu at (37.6, 22.4)
- added R127: 4.7K, Resistor_SMD:R_1206_3216Metric, F.Cu at (36.1, 31.0)
- added R128: 10K, Resistor_SMD:R_0603_1608Metric, F.Cu at (-65.1, 69.4)
- added R129: 220K, Resistor_SMD:R_1206_3216Metric, F.Cu at (-63.6, 65.4)
- added R130: 100K, Resistor_SMD:R_1206_3216Metric, F.Cu at (-63.1, 52.9)
- added R131: 4.7K, Resistor_SMD:R_1206_3216Metric, F.Cu at (-64.6, 61.4)
- added R132: 10K, Resistor_SMD:R_0603_1608Metric, F.Cu at (2.02, 84.6)
- added R133: 220K, Resistor_SMD:R_1206_3216Metric, F.Cu at (3.52, 80.6)
- added R134: 100K, Resistor_SMD:R_1206_3216Metric, F.Cu at (4.03, 68.1)
- added R135: 4.7K, Resistor_SMD:R_1206_3216Metric, F.Cu at (2.52, 76.6)
- added R136: 10K, Resistor_SMD:R_0603_1608Metric, F.Cu at (52.4, 54.2)
- added R137: 220K, Resistor_SMD:R_1206_3216Metric, F.Cu at (53.9, 50.2)
- added R138: 100K, Resistor_SMD:R_1206_3216Metric, F.Cu at (54.4, 37.7)
- added R139: 4.7K, Resistor_SMD:R_1206_3216Metric, F.Cu at (52.9, 46.2)
- added R140: 10K, Resistor_SMD:R_0603_1608Metric, F.Cu at (18.8, 69.4)
- added R141: 220K, Resistor_SMD:R_1206_3216Metric, F.Cu at (20.3, 65.4)
- added R142: 100K, Resistor_SMD:R_1206_3216Metric, F.Cu at (20.8, 52.9)
- added R143: 4.7K, Resistor_SMD:R_1206_3216Metric, F.Cu at (19.3, 61.4)
- added R144: 10K, Resistor_SMD:R_0603_1608Metric, F.Cu at (35.6, 69.4)
- added R145: 220K, Resistor_SMD:R_1206_3216Metric, F.Cu at (37.1, 65.4)
- added R146: 100K, Resistor_SMD:R_1206_3216Metric, F.Cu at (37.6, 52.9)
- added R147: 4.7K, Resistor_SMD:R_1206_3216Metric, F.Cu at (36.1, 61.4)
- added R148: 10K, Resistor_SMD:R_0603_1608Metric, F.Cu at (52.4, 69.4)
- added R149: 220K, Resistor_SMD:R_1206_3216Metric, F.Cu at (53.9, 65.4)
- added R150: 100K, Resistor_SMD:R_1206_3216Metric, F.Cu at (54.4, 52.9)
- added R151: 4.7K, Resistor_SMD:R_1206_3216Metric, F.Cu at (52.9, 61.4)
- added R152: 10K, Resistor_SMD:R_0603_1608Metric, F.Cu at (-65.1, 84.6)
- added R153: 220K, Resistor_SMD:R_1206_3216Metric, F.Cu at (-63.6, 80.6)
- added R154: 100K, Resistor_SMD:R_1206_3216Metric, F.Cu at (-63.1, 68.1)
- added R155: 4.7K, Resistor_SMD:R_1206_3216Metric, F.Cu at (-64.6, 76.6)
- added R156: 10K, Resistor_SMD:R_0603_1608Metric, F.Cu at (-31.6, 84.6)
- added R157: 220K, Resistor_SMD:R_1206_3216Metric, F.Cu at (-30.1, 80.6)
- added R158: 100K, Resistor_SMD:R_1206_3216Metric, F.Cu at (-29.6, 68.1)
- added R159: 4.7K, Resistor_SMD:R_1206_3216Metric, F.Cu at (-31.1, 76.6)
- added R160: 10K, Resistor_SMD:R_0603_1608Metric, F.Cu at (-65.1, 54.2)
- added R161: 220K, Resistor_SMD:R_1206_3216Metric, F.Cu at (-63.6, 50.2)
- added R162: 100K, Resistor_SMD:R_1206_3216Metric, F.Cu at (-63.1, 37.7)
- added R163: 4.7K, Resistor_SMD:R_1206_3216Metric, F.Cu at (-64.6, 46.2)
- added R164: 10K, Resistor_SMD:R_0603_1608Metric, F.Cu at (-31.6, 54.2)
- added R165: 220K, Resistor_SMD:R_1206_3216Metric, F.Cu at (-30.1, 50.2)
- added R166: 100K, Resistor_SMD:R_1206_3216Metric, F.Cu at (-29.6, 37.7)
- added R167: 4.7K, Resistor_SMD:R_1206_3216Metric, F.Cu at (-31.1, 46.2)
- added R168: 10K, Resistor_SMD:R_0603_1608Metric, F.Cu at (35.6, 54.2)
- added R169: 220K, Resistor_SMD:R_1206_3216Metric, F.Cu at (37.1, 50.2)
- added R170: 100K, Resistor_SMD:R_1206_3216Metric, F.Cu at (37.6, 37.7)
- added R171: 4.7K, Resistor_SMD:R_1206_3216Metric, F.Cu at (36.1, 46.2)
- added R172: 10K, Resistor_SMD:R_0603_1608Metric, F.Cu at (-65.1, 38.9)
- added R173: 220K, Resistor_SMD:R_1206_3216Metric, F.Cu at (-63.6, 34.9)
- added R174: 100K, Resistor_SMD:R_1206_3216Metric, F.Cu at (-63.1, 22.4)
- added R175: 4.7K, Resistor_SMD:R_1206_3216Metric, F.Cu at (-64.6, 31.0)
- added R176: 10K, Resistor_SMD:R_0603_1608Metric, F.Cu at (-65.1, 8.49)
- added R177: 220K, Resistor_SMD:R_1206_3216Metric, F.Cu at (-63.6, 4.50)
- added R178: 100K, Resistor_SMD:R_1206_3216Metric, F.Cu at (-63.1, -8.01)
- added R179: 4.7K, Resistor_SMD:R_1206_3216Metric, F.Cu at (-64.6, 0.55)
- added R180: 10K, Resistor_SMD:R_0603_1608Metric, F.Cu at (-31.6, 69.4)
- added R181: 220K, Resistor_SMD:R_1206_3216Metric, F.Cu at (-30.1, 65.4)
- added R182: 100K, Resistor_SMD:R_1206_3216Metric, F.Cu at (-29.6, 52.9)
- added R183: 4.7K, Resistor_SMD:R_1206_3216Metric, F.Cu at (-31.1, 61.4)
- added R184: 10K, Resistor_SMD:R_0603_1608Metric, F.Cu at (-48.3, 23.7)
- added R185: 220K, Resistor_SMD:R_1206_3216Metric, F.Cu at (-46.8, 19.7)
- added R186: 100K, Resistor_SMD:R_1206_3216Metric, F.Cu at (-46.3, 7.21)
- added R187: 4.7K, Resistor_SMD:R_1206_3216Metric, F.Cu at (-47.8, 15.8)
- added R188: 10K, Resistor_SMD:R_0603_1608Metric, F.Cu at (2.02, 99.8)
- added R189: 220K, Resistor_SMD:R_1206_3216Metric, F.Cu at (3.52, 95.8)
- added R190: 100K, Resistor_SMD:R_1206_3216Metric, F.Cu at (4.03, 83.3)
- added R191: 4.7K, Resistor_SMD:R_1206_3216Metric, F.Cu at (2.52, 91.9)
- added R192: 10K, Resistor_SMD:R_0603_1608Metric, F.Cu at (2.02, 23.7)
- added R193: 220K, Resistor_SMD:R_1206_3216Metric, F.Cu at (3.52, 19.7)
- added R194: 100K, Resistor_SMD:R_1206_3216Metric, F.Cu at (4.03, 7.21)
- added R195: 4.7K, Resistor_SMD:R_1206_3216Metric, F.Cu at (2.52, 15.8)
- added R196: 10K, Resistor_SMD:R_0603_1608Metric, F.Cu at (2.02, 69.4)
- added R197: 220K, Resistor_SMD:R_1206_3216Metric, F.Cu at (3.52, 65.4)
- added R198: 100K, Resistor_SMD:R_1206_3216Metric, F.Cu at (4.03, 52.9)
- added R199: 4.7K, Resistor_SMD:R_1206_3216Metric, F.Cu at (2.52, 61.4)
- added R200: 10K, Resistor_SMD:R_0603_1608Metric, F.Cu at (-48.3, 84.6)
- added R201: 220K, Resistor_SMD:R_1206_3216Metric, F.Cu at (-46.8, 80.6)
- added R202: 100K, Resistor_SMD:R_1206_3216Metric, F.Cu at (-46.3, 68.1)
- added R203: 4.7K, Resistor_SMD:R_1206_3216Metric, F.Cu at (-47.8, 76.6)
- added R204: 10K, Resistor_SMD:R_0603_1608Metric, F.Cu at (-65.1, 115.0)
- added R205: 220K, Resistor_SMD:R_1206_3216Metric, F.Cu at (-63.6, 111.0)
- added R206: 100K, Resistor_SMD:R_1206_3216Metric, F.Cu at (-63.1, 98.5)
- added R207: 4.7K, Resistor_SMD:R_1206_3216Metric, F.Cu at (-64.6, 107.1)
- added R208: 10K, Resistor_SMD:R_0603_1608Metric, F.Cu at (2.02, 8.49)
- added R209: 220K, Resistor_SMD:R_1206_3216Metric, F.Cu at (3.52, 4.50)
- added R210: 100K, Resistor_SMD:R_1206_3216Metric, F.Cu at (4.03, -8.01)
- added R211: 4.7K, Resistor_SMD:R_1206_3216Metric, F.Cu at (2.52, 0.55)
- added R212: 10K, Resistor_SMD:R_0603_1608Metric, F.Cu at (18.8, 84.6)
- added R213: 220K, Resistor_SMD:R_1206_3216Metric, F.Cu at (20.3, 80.6)
- added R214: 100K, Resistor_SMD:R_1206_3216Metric, F.Cu at (20.8, 68.1)
- added R215: 4.7K, Resistor_SMD:R_1206_3216Metric, F.Cu at (19.3, 76.6)
- added R216: 10K, Resistor_SMD:R_0603_1608Metric, F.Cu at (-31.6, 23.7)
- added R217: 220K, Resistor_SMD:R_1206_3216Metric, F.Cu at (-30.1, 19.7)
- added R218: 100K, Resistor_SMD:R_1206_3216Metric, F.Cu at (-29.6, 7.21)
- added R219: 4.7K, Resistor_SMD:R_1206_3216Metric, F.Cu at (-31.1, 15.8)
- added R220: 10K, Resistor_SMD:R_0603_1608Metric, F.Cu at (18.8, 23.7)
- added R221: 220K, Resistor_SMD:R_1206_3216Metric, F.Cu at (20.3, 19.7)
- added R222: 100K, Resistor_SMD:R_1206_3216Metric, F.Cu at (20.8, 7.21)
- added R223: 4.7K, Resistor_SMD:R_1206_3216Metric, F.Cu at (19.3, 15.8)
- added R224: 10K, Resistor_SMD:R_0603_1608Metric, F.Cu at (-14.8, 23.7)
- added R225: 220K, Resistor_SMD:R_1206_3216Metric, F.Cu at (-13.3, 19.7)
- added R226: 100K, Resistor_SMD:R_1206_3216Metric, F.Cu at (-12.8, 7.21)
- added R227: 4.7K, Resistor_SMD:R_1206_3216Metric, F.Cu at (-14.3, 15.8)
- added R228: 10K, Resistor_SMD:R_0603_1608Metric, F.Cu at (-48.3, 115.0)
- added R229: 220K, Resistor_SMD:R_1206_3216Metric, F.Cu at (-46.8, 111.0)
- added R230: 100K, Resistor_SMD:R_1206_3216Metric, F.Cu at (-46.3, 98.5)
- added R231: 4.7K, Resistor_SMD:R_1206_3216Metric, F.Cu at (-47.8, 107.1)
- added R232: 10K, Resistor_SMD:R_0603_1608Metric, F.Cu at (18.8, 38.9)
- added R233: 220K, Resistor_SMD:R_1206_3216Metric, F.Cu at (20.3, 34.9)
- added R234: 100K, Resistor_SMD:R_1206_3216Metric, F.Cu at (20.8, 22.4)
- added R235: 4.7K, Resistor_SMD:R_1206_3216Metric, F.Cu at (19.3, 31.0)
- added R236: 10K, Resistor_SMD:R_0603_1608Metric, F.Cu at (-31.6, 38.9)
- added R237: 220K, Resistor_SMD:R_1206_3216Metric, F.Cu at (-30.1, 34.9)
- added R238: 100K, Resistor_SMD:R_1206_3216Metric, F.Cu at (-29.6, 22.4)
- added R239: 4.7K, Resistor_SMD:R_1206_3216Metric, F.Cu at (-31.1, 31.0)
- added R240: 10K, Resistor_SMD:R_0603_1608Metric, F.Cu at (35.6, 84.6)
- added R241: 220K, Resistor_SMD:R_1206_3216Metric, F.Cu at (37.1, 80.6)
- added R242: 100K, Resistor_SMD:R_1206_3216Metric, F.Cu at (37.6, 68.1)
- added R243: 4.7K, Resistor_SMD:R_1206_3216Metric, F.Cu at (36.1, 76.6)
- added R244: 10K, Resistor_SMD:R_0603_1608Metric, F.Cu at (-48.3, 8.49)
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Connections:
- C1 pad 1: Net-(C1-Pad1) -> +12V
- C1 pad 2: Net-(C1-Pad2) -> GND
- C10 pad 1: GND -> +5V
- C10 pad 2: VCC -> GND
- C2 pad 1: Net-(C2-Pad1) -> +12V
- C2 pad 2: Net-(C2-Pad2) -> GND
- C3 pad 1: Net-(C3-Pad1) -> +5V
- C3 pad 2: Net-(C3-Pad2) -> GND
- C4 pad 1: Net-(C4-Pad1) -> +5V
- C4 pad 2: Net-(C4-Pad2) -> GND
- C5 pad 1: Net-(C5-Pad1) -> +3V3
- C5 pad 2: Net-(C5-Pad2) -> GND
- C6 pad 1: Net-(C6-Pad1) -> /VUSB
- C6 pad 2: Net-(C6-Pad2) -> GND
- C7 pad 1: Net-(C7-Pad1) -> +5V
- C7 pad 2: Net-(C7-Pad2) -> GND
- C8 pad 1: Net-(C8-Pad1) -> +5V
- C8 pad 2: Net-(C8-Pad2) -> GND
- C9 pad 1: GND -> +5V
- C9 pad 2: VCC -> GND
- J1 pad 1: VCC -> HT
- J2 pad 1: AO0 -> +5V
- J2 pad 2: AO1 -> /K_ADDR_LED_5V
- J2 pad 3: AO2 -> /K_CLK_5V
- J2 pad 4: AO3 -> /K_RST_5V
- J2 pad 5: AO4 -> GND
- J3 pad 1: Net-(J3-Pad1) -> GND
- J3 pad 2: Net-(J3-Pad2) -> unconnected-(J3-Pin_2-Pad2)
- J3 pad 3: Net-(J3-Pad3) -> unconnected-(J3-Pin_3-Pad3)
- J3 pad 4: Net-(J3-Pad4) -> +12V
- J4 pad 1: VCC -> HT
- J5 pad 1: KO0 -> +3V3
- J5 pad 2: KO1 -> Net-(J5-SWDIO)
- J5 pad 3: KO2 -> /RST
- J5 pad 4: KO3 -> Net-(J5-SWCLK)
- J5 pad 5: KO4 -> GND
- J5 pad 6: KO5 -> unconnected-(J5-SWO-Pad6)
- Q1 pad 1: Net-(Q1-Pad1) -> Net-(D9-K)
- Q1 pad 2: Net-(C1-Pad2) -> Net-(D9-A)
- Q10 pad 1: Net-(Q10-Pad1) -> Net-(Q10-B)
- Q10 pad 3: Net-(Q10-Pad3) -> Net-(D17-K)
- Q11 pad 1: Net-(Q11-Pad1) -> Net-(D19-K)
- Q11 pad 2: GND -> Net-(D19-A)
- Q11 pad 3: Net-(Q11-Pad3) -> HT
- Q12 pad 1: Net-(Q12-Pad1) -> Net-(Q12-B)
- Q12 pad 3: Net-(Q12-Pad3) -> Net-(D19-K)
- Q13 pad 1: Net-(Q13-Pad1) -> Net-(D21-K)
- Q13 pad 2: GND -> Net-(D21-A)
- Q13 pad 3: Net-(Q13-Pad3) -> HT
- Q14 pad 1: Net-(Q14-Pad1) -> Net-(Q14-B)
- Q14 pad 3: Net-(Q14-Pad3) -> Net-(D21-K)
- Q15 pad 1: Net-(Q15-Pad1) -> Net-(D23-K)
- Q15 pad 2: GND -> Net-(D23-A)
- Q15 pad 3: Net-(Q15-Pad3) -> HT
- Q16 pad 1: Net-(Q16-Pad1) -> Net-(Q16-B)
- Q16 pad 3: Net-(Q16-Pad3) -> Net-(D23-K)
- Q17 pad 1: Net-(Q17-Pad1) -> Net-(D25-K)
- Q17 pad 2: GND -> Net-(D25-A)
- Q17 pad 3: KO0 -> HT
- Q18 pad 1: Net-(Q18-Pad1) -> Net-(Q18-B)
- Q18 pad 3: KO1 -> Net-(D25-K)
- Q19 pad 1: Net-(Q19-Pad1) -> Net-(D27-K)
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Routing:
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- removed copper zone on B.Cu, net GND
- removed copper zone on F.Cu, net GND
- removed copper zone on B.Cu, net HT
- removed copper zone on F.Cu, net HT
Other:
- board outline removed
- net class Default removed
- board text removed: "1 2 3 4 5 6 7 8 ANODE"
- board text removed: "8 7 6 5 4 3 2 1 CATHODE"
- board text removed: "A0"
- board text removed: "A1"
- board text removed: "A2"
- board text removed: "A3"
- board text removed: "A4"
- board text removed: "A5"
- board text removed: "A6"
- board text removed: "A7"
- board text removed: "ANODE 1 2 3 4 5 6 7 8"
- board text removed: "AS"
- board text removed: "CATHODE 8 7 6 5 4 3 2 1"
- board text removed: "Gnd"
- board text removed: "HV"
- board text removed: "K0"
- board text removed: "K1"
- board text removed: "K2"
- board text removed: "K3"
- board text removed: "K4"
- board text removed: "K5"
- board text removed: "K6"
- board text removed: "K7"
- board text removed: "KS"
- board text removed: "Vcc"
- board text removed: "driver"
- board text removed: "hackaday.io/muth"
- board text removed: "ИГГ_ octal"

Commit message: Pretty far on the anode layout
Parts:
- moved R176 283.1 mm to (194.5, 121.3), turned to 90 degrees
- moved C70 279.9 mm to (194.5, 109.8)
- moved R178 279.2 mm to (192.0, 105.3)
- moved D90 279.0 mm to (190.5, 109.3)
- moved R177 279.0 mm to (191.5, 117.3)
- moved R179 278.9 mm to (190.5, 113.3)
- moved Q81 278.8 mm to (194.0, 113.8)
- moved D89 278.5 mm to (195.0, 117.3)
- moved Q82 277.6 mm to (191.4, 120.8)
- moved R228 271.5 mm to (210.5, 33.2), turned to 90 degrees
- moved R244 270.9 mm to (218.5, 55.2), turned to 90 degrees
- moved C83 268.1 mm to (210.5, 21.7)
- moved R204 267.7 mm to (202.5, 121.3), turned to 90 degrees
- moved D115 267.5 mm to (211.0, 29.2)
- moved C87 267.5 mm to (218.5, 43.7)
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Routing:
- net /AO61: track 0.54 -> 99.4 mm
- net /AO62: track 0.54 -> 78.2 mm
- net /AO63: track 0.54 -> 58.1 mm, vias 1 -> 2
- net /AO64: track 0.54 -> 35.0 mm
- net /AO59: track 0.54 -> 33.8 mm
- net HT: track 338.1 -> 363.4 mm, vias 62 -> 63
- net GND: track 67.2 -> 51.0 mm, vias 62 -> 63
- net /AO60: track 0.54 -> 10.7 mm
- net Net-(D123-A): track 11.5 -> 2.04 mm, vias 0 -> 2
- net Net-(D13-K): track 0.00 -> 9.12 mm
- net Net-(D13-A): track 0.00 -> 8.51 mm, vias 0 -> 2
- net Net-(D11-A): track 0.00 -> 6.96 mm, vias 0 -> 2
- net Net-(D11-K): track 0.00 -> 6.74 mm
- net Net-(D12-K): track 0.00 -> 4.84 mm
- net Net-(D14-K): track 0.00 -> 4.74 mm
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Other:
- board outline added: 162.5 x 147 mm
- copper layers 2 -> 4
- rule pad_to_mask_clearance: 0.0254 -> 0

Commit message: Added design files for the kathode, mods to the anode board
Parts:
- moved H1 146.6 mm to (13.2, 210.0)
- moved C19 132.9 mm to (68.0, 195.1)
- moved C20 132.9 mm to (68.0, 197.6)
- moved C21 132.9 mm to (68.0, 200.1)
- moved C22 132.9 mm to (68.0, 202.6)
- moved C23 132.9 mm to (68.0, 205.1)
- moved D1 132.9 mm to (25.9, 217.6)
- moved R12 132.9 mm to (80.1, 195.1)
- moved R13 132.9 mm to (80.1, 197.6)
- moved R14 132.9 mm to (80.1, 200.1)
- moved R15 132.9 mm to (80.1, 202.6)
- moved U12 132.9 mm to (121.1, 202.6)
- moved C1 132.9 mm to (38.5, 216.3)
- moved C10 132.9 mm to (42.5, 218.8)
- moved C11 132.9 mm to (64.0, 195.1)
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Routing:
- net /AO6: track 0.79 -> 124.1 mm
- net /AO16: track 0.79 -> 123.2 mm
- net /AO11: track 0.79 -> 121.5 mm
- net /AO21: track 0.79 -> 120.6 mm
- net /AO26: track 0.79 -> 113.7 mm
- net /AI45: track 0.67 -> 113.2 mm, vias 1 -> 2
- net /AO31: track 0.79 -> 112.1 mm
- net /AI60: track 0.67 -> 111.1 mm, vias 1 -> 2
- net /AI55: track 0.67 -> 109.9 mm, vias 1 -> 2
- net /AI50: track 0.67 -> 108.1 mm, vias 1 -> 2
- net /AO36: track 0.79 -> 106.6 mm
- net /AO41: track 0.79 -> 105.6 mm
- net /AO8: track 0.79 -> 101.4 mm
- net /AO46: track 0.79 -> 101.3 mm
- net /AO12: track 0.79 -> 100.7 mm
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- added copper zone on B.Cu, net GND
- added copper zone on In1.Cu, net HT
Other:
- outline, holes or cut-outs redrawn
