File: IGGDriver/IGGDriver/IP2368.kicad_sch (KiCad schematic)
At the start: 23 parts, among them U16 IP2326

Commit message: progress!
Parts:
- removed C101: C, symbol Device:C
- removed R281: R, symbol Device:R
- added C15: 22u, Capacitor_SMD:C_1206_3216Metric, symbol Device:C
- added JP1: BAT_EN, symbol Jumper:SolderJumper_2_Open
- added JP14: Jumper_2_Bridged, symbol Jumper:Jumper_2_Bridged
- added SW7: PWR, symbol Switch:SW_SPST
- C95, C96, C99: footprint (none) -> Capacitor_SMD:C_0603_1608Metric; LCSC (none) -> C14663
- L2: footprint (none) -> Inductor_SMD:L_1008_2520Metric; LCSC (none) -> C488330
- R272, R275, R276: footprint (none) -> Resistor_SMD:R_0603_1608Metric; LCSC (none) -> C23231
- R273, R274, R277: footprint (none) -> Resistor_SMD:R_0603_1608Metric; LCSC (none) -> C25803
- R278: footprint (none) -> Resistor_SMD:R_0603_1608Metric; LCSC (none) -> C22962
- R282: value 5.1K -> DNP; footprint (none) -> Resistor_SMD:R_0603_1608Metric
- U16: footprint MODULE -> Package_DFN_QFN:QFN-24-1EP_4x4mm_P0.5mm_EP2.6x2.6mm_ThermalVias; LCSC (none) -> C2832094
Connections:
- net GND: now also C15.2, JP1.1 (A), SW7.1 (A); no longer BT1.2 (-)
- net V_USB: now also JP14.2 (B)
- net at U16.13 (VIN): now also C15.1, JP14.1 (A)
- net BAT_MID: now reaches BT1.1 (+), BT2.2 (-), C95.2, C96.1, R278.2
- new net: BT1.2 (-), JP1.2 (B), SW7.2 (B)

Commit message: Commit to xfer to other computer
Parts:
- removed JP1: BAT_EN, symbol Jumper:SolderJumper_2_Open
- removed SW7: PWR, symbol Switch:SW_SPST
Connections:
- net GND: now also BT1.2 (-)
- net EN: no longer names the net of R277.2, U16.12 (EN)

Commit message: Push to other computer to edit footprint
Parts:
- removed JP14: Jumper_2_Bridged, symbol Jumper:Jumper_2_Bridged
Connections:
- net GND: now also U16.25 (PAD); no longer U16. (PAD)
- net V_USB: now also C15.1, U16.13 (VIN)
Changed lines of the file:
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@@
-	(wire
-		(pts
-			(xy 120.65 40.64) (xy 120.65 43.18)
-		)
-		(stroke
-			(width 0)
-			(type default)
-		)
-	)
 	(wire
 		(pts
@@
 	(wire
 		(pts
-			(xy 120.65 29.21) (xy 120.65 30.48)
+			(xy 120.65 29.21) (xy 120.65 43.18)
 		)
 		(stroke
@@
 		(pin "22"
 		)
-		(pin ""
+		(pin "25"
 		)
 		(instances
@@
 					(unit 1)
 				)
-			)
-		)
-	)
-	(symbol
-		(lib_id "Jumper:Jumper_2_Bridged")
-		(at 120.65 35.56 90)
-		(unit 1)
-		(exclude_from_sim yes)
-		(in_bom yes)
-		(on_board yes)
-		(dnp no)
-		(fields_autoplaced yes)
-		(property "Reference" "JP14"
-			(at 121.92 34.2899 90)
-			(effects
-				(font
-					(size 1.27 1.27)
-				)
-				(justify right)
-			)
-		)
-		(property "Value" "Jumper_2_Bridged"
-			(at 121.92 36.8299 90)
-			(effects
-				(font
-					(size 1.27 1.27)
-				)
-				(justify right)
-			)
-		)
-		(property "Footprint" ""
-			(at 120.65 35.56 0)
-			(effects
-				(font
-					(size 1.27 1.27)
-				)
-				(hide yes)
-			)
-		)
-		(property "Datasheet" "~"
-			(at 120.65 35.56 0)
-			(effects
-				(font
-					(size 1.27 1.27)
-				)
-				(hide yes)
-			)
-		)
-		(property "Description" "Jumper, 2-pole, closed/bridged"
-			(at 120.65 35.56 0)
-			(effects
-				(font
-					(size 1.27 1.27)
-				)
-				(hide yes)
-			)
-		)
-		(pin "1"
-		)
-		(pin "2"
-		)
-		(instances
-			(project "IGGDriver"
-				(path "/42dcdc8e-b1dc-4d4c-b3c7-96447ce841be/ed6672d7-92eb-40ce-b4cc-e5b4f765c723"
-					(reference "JP14")
-					(unit 1)
-				)

Commit message: RTM
Parts:
- added J3: Conn_01x03, Connector_JST:JST_XH_B3B-XH-AM_1x03_P2.50mm_Vertical, symbol Connector_Generic:Conn_01x03
Connections:
- net BAT_MID: now also J3.2 (Pin_2)
- net GND: now also J3.3 (Pin_3)
- net at BT2.1 (+), C94.1, C95.1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: now also J3.1 (Pin_1)
Changed lines of the file:
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@@
+	)
+	(junction
+		(at 213.36 69.85)
+		(diameter 0)
+		(color 0 0 0 0)
 	)
 	(junction
@@
 	(wire
 		(pts
+			(xy 224.79 78.74) (xy 224.79 69.85)
+		)
+		(stroke
+			(width 0)
+			(type default)
+		)
+	)
+	(wire
+		(pts
 			(xy 140.97 69.85) (xy 147.32 69.85)
 		)
@@
 	(wire
 		(pts
+			(xy 231.14 81.28) (xy 223.52 81.28)
+		)
+		(stroke
+			(width 0)
+			(type default)
+		)
+	)
+	(wire
+		(pts
+			(xy 231.14 78.74) (xy 224.79 78.74)
+		)
+		(stroke
+			(width 0)
+			(type default)
+		)
+	)
+	(wire
+		(pts
 			(xy 179.07 85.09) (xy 179.07 74.93)
 		)
@@
 	(wire
 		(pts
+			(xy 223.52 85.09) (xy 203.2 85.09)
+		)
+		(stroke
+			(width 0)
+			(type default)
+		)
+	)
+	(wire
+		(pts
 			(xy 213.36 82.55) (xy 213.36 86.36)
 		)
@@
 	(wire
 		(pts
+			(xy 223.52 81.28) (xy 223.52 85.09)
+		)
+		(stroke
+			(width 0)
+			(type default)
+		)
+	)
+	(wire
+		(pts
 			(xy 88.9 87.63) (xy 95.25 87.63)
 		)
@@
 		(pts
 			(xy 115.57 105.41) (xy 115.57 107.95)
+		)
+		(stroke
+			(width 0)
+			(type default)
+		)
+	)
+	(wire
+		(pts
+			(xy 224.79 69.85) (xy 213.36 69.85)
 		)
 		(stroke
@@
 					(unit 1)
 				)
+			)
+		)
+	)
+	(symbol
+		(lib_id "Connector_Generic:Conn_01x03")
+		(at 236.22 81.28 0)
+		(unit 1)
+		(exclude_from_sim no)
+		(in_bom yes)
+		(on_board yes)
+		(dnp no)
+		(fields_autoplaced yes)
+		(property "Reference" "J3"
+			(at 238.76 80.0099 0)
+			(effects
+				(font
+					(size 1.27 1.27)
+				)
+				(justify left)
+			)
+		)
+		(property "Value" "Conn_01x03"
+			(at 238.76 82.5499 0)
+			(effects
+				(font
+					(size 1.27 1.27)
+				)
+				(justify left)
+			)
+		)
+		(property "Footprint" "Connector_JST:JST_XH_B3B-XH-AM_1x03_P2.50mm_Vertical"
+			(at 236.22 81.28 0)
+			(effects
+				(font
+					(size 1.27 1.27)
+				)
+				(hide yes)
+			)
+		)
+		(property "Datasheet" "~"
+			(at 236.22 81.28 0)
+			(effects
+				(font
+					(size 1.27 1.27)
+				)
+				(hide yes)
+			)
+		)
+		(property "Description" "Generic connector, single row, 01x03, script generated (kicad-library-utils/schlib/autogen/connector/)"
+			(at 236.22 81.28 0)
+			(effects
+				(font
+					(size 1.27 1.27)
+				)
+				(hide yes)
+			)
+		)
+		(property "LCSC" ""
+			(at 236.22 81.28 0)
+			(effects
+				(font
+					(size 1.27 1.27)
+				)
+				(hide yes)
+			)
+		)
+		(pin "3"
+		)
+		(pin "2"
+		)
+		(pin "1"
+		)
+		(instances
+			(project "IGGDriver"
+				(path "/42dcdc8e-b1dc-4d4c-b3c7-96447ce841be/ed6672d7-92eb-40ce-b4cc-e5b4f765c723"
+					(reference "J3")
+					(unit 1)
+				)
+			)
+		)
+	)
+	(symbol
+		(lib_id "power:GND")
+		(at 231.14 83.82 0)
+		(unit 1)
+		(exclude_from_sim no)
+		(in_bom yes)
+		(on_board yes)
+		(dnp no)
+		(fields_autoplaced yes)
+		(property "Reference" "#PWR052"
+			(at 231.14 90.17 0)
+			(effects
+				(font
+					(size 1.27 1.27)
+				)
+				(hide yes)
+			)
+		)
+		(property "Value" "GND"
+			(at 231.14 88.9 0)
+			(effects
+				(font
+					(size 1.27 1.27)
+				)
+			)
+		)
+		(property "Footprint" ""
+			(at 231.14 83.82 0)
+			(effects
+				(font
+					(size 1.27 1.27)
+				)
+				(hide yes)
+			)
+		)
+		(property "Datasheet" ""
+			(at 231.14 83.82 0)
+			(effects
+				(font
+					(size 1.27 1.27)
+				)
+				(hide yes)
+			)
+		)
+		(property "Description" "Power symbol creates a global label with name \"GND\" , ground"
+			(at 231.14 83.82 0)
+			(effects
+				(font
+					(size 1.27 1.27)
+				)
+				(hide yes)
+			)
+		)
+		(pin "1"
+		)
+		(instances
+			(project "IGGDriver"
+				(path "/42dcdc8e-b1dc-4d4c-b3c7-96447ce841be/ed6672d7-92eb-40ce-b4cc-e5b4f765c723"
+					(reference "#PWR052")
+					(unit 1)
+				)
