File: IGGDriver/IGGDriver/TPS5430.kicad_sch (KiCad schematic)
At the start: 8 parts, among them U18 TPS5430DDA

Commit message: Commit to xfer to other computer
Other:
- note added: "Float to enable"
Changed lines of the file:
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@@
+		)
+	)
+	(text "Float to enable"
+		(exclude_from_sim no)
+		(at 87.63 104.902 0)
+		(effects
+			(font
+				(size 1.27 1.27)
+			)
 		)
 	)

Commit message: RTM
Parts:
- L4: LCSC C408533 -> C408533
Changed lines of the file:
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@@
 			)
 		)
-		(property "LCSC" "    C408533"
+		(property "LCSC" " C408533"
 			(at 132.08 85.09 90)
 			(effects
