File: IGGDriver/IGGDriver/anode.kicad_sch (KiCad schematic)
At the start: 9 parts, among them Q100 Q_NPN_BEC, Q99 Q_NPN_BEC

Commit message: combined the pcbs, now to relayout. :(
Parts:
- renumbered C79 to C49, D107 to D47, D108 to D48, Q99 to Q39, Q100 to Q40, R212 to R92, R213 to R93, R214 to R94, R215 to R95

Commit message: almost done
Parts:
- D47, D48: LCSC C896450 -> C110231
Changed lines of the file:
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@@
 			)
 		)
-		(property "LCSC" "C896450"
+		(property "LCSC" "C110231"
 			(at 137.16 102.87 90)
 			(effects
@@
 			)
 		)
-		(property "LCSC" "C896450"
+		(property "LCSC" "C110231"
 			(at 142.24 102.87 90)
 			(effects

Commit message: Push to other computer to edit footprint
Parts:
- renumbered C49 to C79, D47 to D107, D48 to D108, Q40 to Q100, Q39 to Q99, R92 to R212, R93 to R213, R94 to R214, R95 to R215

Commit message: RTM
Parts:
- renumbered C79 to C49, D107 to D47, D108 to D48, Q99 to Q39, Q100 to Q40, R212 to R92, R213 to R93, R214 to R94, R215 to R95
