File: IGGDriver/IGGDriver/kathodeDriver/kathodeDriver.kicad_sch (KiCad schematic)
At the start: 232 parts, among them J1001 Conn_01x05, J1002 Conn_01x02, Q1001 Q_NPN_BEC, Q1002 Q_NPN_BEC, Q1003 Q_NPN_BEC, Q1004 Q_NPN_BEC, Q1005 Q_NPN_BEC, Q1006 Q_NPN_BEC, Q1007 Q_NPN_BEC, Q1008 Q_NPN_BEC, Q1009 Q_NPN_BEC, Q1010 Q_NPN_BEC, Q1011 Q_NPN_BEC, Q1012 Q_NPN_BEC, Q1013 Q_NPN_BEC, Q1014 Q_NPN_BEC, Q1015 Q_NPN_BEC, Q1016 Q_NPN_BEC, Q1017 Q_NPN_BEC, Q1018 Q_NPN_BEC, Q1019 Q_NPN_BEC, Q1020 Q_NPN_BEC, Q1021 Q_NPN_BEC, Q1022 Q_NPN_BEC, Q1023 Q_NPN_BEC, Q1024 Q_NPN_BEC, Q1025 Q_NPN_BEC, Q1026 Q_NPN_BEC, Q1027 Q_NPN_BEC, Q1028 Q_NPN_BEC, Q1029 Q_NPN_BEC, Q1030 Q_NPN_BEC, Q1031 Q_NPN_BEC, Q1032 Q_NPN_BEC, Q1033 Q_NPN_BEC, Q1034 Q_NPN_BEC, Q1035 Q_NPN_BEC, Q1036 Q_NPN_BEC, Q1037 Q_NPN_BEC, Q1038 Q_NPN_BEC, Q1039 Q_NPN_BEC, Q1040 Q_NPN_BEC, Q1041 Q_NPN_BEC, Q1042 Q_NPN_BEC, Q1043 Q_NPN_BEC, Q1044 Q_NPN_BEC, Q1045 Q_NPN_BEC, Q1046 Q_NPN_BEC, Q1047 Q_NPN_BEC, Q1048 Q_NPN_BEC, Q1049 Q_NPN_BEC, Q1050 Q_NPN_BEC, Q1051 Q_NPN_BEC, Q1052 Q_NPN_BEC, Q1053 Q_NPN_BEC, Q1054 Q_NPN_BEC, Q1055 Q_NPN_BEC, Q1056 Q_NPN_BEC, Q1057 Q_NPN_BEC, Q1058 Q_NPN_BEC, Q1059 Q_NPN_BEC, Q1060 Q_NPN_BEC, Q1061 Q_NPN_BEC, Q1062 Q_NPN_BEC, Q1063 Q_NPN_BEC, Q1064 Q_NPN_BEC, U1001 74AUP1G32, U1002 4017, U1003 4081, U1004 4081, U1005 4017, U1006 4017, U1007 4017, U1008 4017, U1009 4017, U1011 4017, U1012 4017

Commit message: combined the pcbs, now to relayout. :(
Parts:
- U13: renamed from U1010; footprint IGG1:IGG1 -> IGG1:IGG1-All; symbol IGG1:IGG1-64 -> IGG1:IGG1-64-All
Changed lines of the file:
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@@
 	)
 	(symbol
-		(lib_id "IGG1:IGG1-64")
+		(lib_id "IGG1:IGG1-64-All")
 		(at 556.26 62.23 0)
 		(unit 1)
@@
 		(dnp no)
 		(fields_autoplaced yes)
-		(property "Reference" "U1010"
+		(property "Reference" "U13"
 			(at 561.34 133.3499 0)
 			(effects
@@
 			)
 		)
-		(property "Footprint" "IGG1:IGG1"
+		(property "Footprint" "IGG1:IGG1-All"
 			(at 556.26 62.23 0)
 			(effects
@@
 		)
 		(pin "16"
+		)
+		(pin "78"
+		)
+		(pin "72"
+		)
+		(pin "67"
+		)
+		(pin "125"
+		)
+		(pin "119"
+		)
+		(pin "122"
+		)
+		(pin "83"
+		)
+		(pin "77"
+		)
+		(pin "102"
+		)
+		(pin "65"
+		)
+		(pin "88"
+		)
+		(pin "84"
+		)
+		(pin "121"
+		)
+		(pin "101"
+		)
+		(pin "69"
+		)
+		(pin "127"
+		)
+		(pin "107"
+		)
+		(pin "111"
+		)
+		(pin "114"
+		)
+		(pin "82"
+		)
+		(pin "103"
+		)
+		(pin "100"
+		)
+		(pin "106"
+		)
+		(pin "99"
+		)
+		(pin "75"
+		)
+		(pin "66"
+		)
+		(pin "105"
+		)
+		(pin "116"
+		)
+		(pin "123"
+		)
+		(pin "112"
+		)
+		(pin "70"
+		)
+		(pin "113"
+		)
+		(pin "92"
+		)
+		(pin "74"
+		)
+		(pin "115"
+		)
+		(pin "126"
+		)
+		(pin "73"
+		)
+		(pin "79"
+		)
+		(pin "110"
+		)
+		(pin "93"
+		)
+		(pin "76"
+		)
+		(pin "95"
+		)
+		(pin "96"
+		)
+		(pin "104"
+		)
+		(pin "91"
+		)
+		(pin "68"
+		)
+		(pin "97"
+		)
+		(pin "98"
+		)
+		(pin "120"
+		)
+		(pin "118"
+		)
+		(pin "94"
+		)
+		(pin "124"
+		)
+		(pin "71"
+		)
+		(pin "108"
+		)
+		(pin "89"
+		)
+		(pin "85"
+		)
+		(pin "81"
+		)
+		(pin "109"
+		)
+		(pin "90"
+		)
+		(pin "87"
+		)
+		(pin "86"
+		)
+		(pin "80"
+		)
+		(pin "128"
+		)
+		(pin "117"
 		)
 		(instances
 			(project "IGGDriver"
 				(path "/42dcdc8e-b1dc-4d4c-b3c7-96447ce841be/2fcadc02-6b88-411f-b68e-dd3f4c7cfe83"
-					(reference "U1010")
+					(reference "U13")
 					(unit 1)
 				)

Commit message: progress!
Parts:
- removed D1001, D1002, D1003, D1004, D1005, D1006: SK6812, LED_SMD:LED_SK6812_PLCC4_5.0x5.0mm_P3.2mm, symbol LED:SK6812
- removed J1001: Conn_01x05, Connector_JST:JST_XH_B4B-XH-AM_1x05_P2.50mm_Vertical, symbol Connector_Generic:Conn_01x05
Connections:
- net RESET_COUNT renamed RESET

Commit message: Push to other computer to edit footprint
Parts:
- removed H1001, H1002: MountingHole, Mounting_Wuerth:Mounting_Wuerth_WA-SMSI-M3_H2mm_9774020360, symbol Mechanical:MountingHole
Changed lines of the file:
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@@
-	)
-	(symbol
-		(lib_id "Mechanical:MountingHole")
-		(at 575.31 278.13 0)
-		(unit 1)
-		(exclude_from_sim yes)
-		(in_bom no)
-		(on_board yes)
-		(dnp no)
-		(fields_autoplaced yes)
-		(property "Reference" "H1002"
-			(at 577.85 276.8599 0)
-			(effects
-				(font
-					(size 1.27 1.27)
-				)
-				(justify left)
-			)
-		)
-		(property "Value" "MountingHole"
-			(at 577.85 279.3999 0)
-			(effects
-				(font
-					(size 1.27 1.27)
-				)
-				(justify left)
-			)
-		)
-		(property "Footprint" "Mounting_Wuerth:Mounting_Wuerth_WA-SMSI-M3_H2mm_9774020360"
-			(at 575.31 278.13 0)
-			(effects
-				(font
-					(size 1.27 1.27)
-				)
-				(hide yes)
-			)
-		)
-		(property "Datasheet" "~"
-			(at 575.31 278.13 0)
-			(effects
-				(font
-					(size 1.27 1.27)
-				)
-				(hide yes)
-			)
-		)
-		(property "Description" "Mounting Hole without connection"
-			(at 575.31 278.13 0)
-			(effects
-				(font
-					(size 1.27 1.27)
-				)
-				(hide yes)
-			)
-		)
-		(instances
-			(project "IGGDriver"
-				(path "/42dcdc8e-b1dc-4d4c-b3c7-96447ce841be/2fcadc02-6b88-411f-b68e-dd3f4c7cfe83"
-					(reference "H1002")
-					(unit 1)
-				)
-			)
-			(project "kathodeDriver"
-				(path "/f2c72e81-6fe3-4213-8891-e652083dbd6a"
-					(reference "H1002")
-					(unit 1)
-				)
-			)
-		)
 	)
 	(symbol
@@
 					(unit 1)
 				)
-			)
-		)
-	)
-	(symbol
-		(lib_id "Mechanical:MountingHole")
-		(at 575.31 273.05 0)
-		(unit 1)
-		(exclude_from_sim yes)
-		(in_bom no)
-		(on_board yes)
-		(dnp no)
-		(fields_autoplaced yes)
-		(property "Reference" "H1001"
-			(at 577.85 271.7799 0)
-			(effects
-				(font
-					(size 1.27 1.27)
-				)
-				(justify left)
-			)
-		)
-		(property "Value" "MountingHole"
-			(at 577.85 274.3199 0)
-			(effects
-				(font
-					(size 1.27 1.27)
-				)
-				(justify left)
-			)
-		)
-		(property "Footprint" "Mounting_Wuerth:Mounting_Wuerth_WA-SMSI-M3_H2mm_9774020360"
-			(at 575.31 273.05 0)
-			(effects
-				(font
-					(size 1.27 1.27)
-				)
-				(hide yes)
-			)
-		)
-		(property "Datasheet" "~"
-			(at 575.31 273.05 0)
-			(effects
-				(font
-					(size 1.27 1.27)
-				)
-				(hide yes)
-			)
-		)
-		(property "Description" "Mounting Hole without connection"
-			(at 575.31 273.05 0)
-			(effects
-				(font
-					(size 1.27 1.27)
-				)
-				(hide yes)
-			)
-		)
-		(instances
-			(project "IGGDriver"
-				(path "/42dcdc8e-b1dc-4d4c-b3c7-96447ce841be/2fcadc02-6b88-411f-b68e-dd3f4c7cfe83"
-					(reference "H1001")
-					(unit 1)
-				)
-			)
-			(project "kathodeDriver"
-				(path "/f2c72e81-6fe3-4213-8891-e652083dbd6a"
-					(reference "H1001")
-					(unit 1)
-				)

Commit message: RTM
Parts:
- removed D1008: LED, LED_SMD:LED_0603_1608Metric, symbol Device:LED
- removed R1002: 1K, Resistor_SMD:R_0603_1608Metric, symbol Device:R

Commit message: Added mechanicDDDDl stuff, case, etc
Parts:
- U1001: LCSC C7470 -> C7470
Changed lines of the file:
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@@
 			)
 		)
-		(property "LCSC" "C7470	"
+		(property "LCSC" "C7470"
 			(at 199.39 411.48 0)
 			(effects
